File: LP_and_HS_LVDS_to_SLVS.sch (KiCad schematic (older format))
At the start: 1 part

Commit message: just commit
Parts:
- added R?: 4.7K, Resistors_SMD:R_0805, symbol Device:R
Connections:
- net labels added: SWITCH_SEL_VADJ, SWITCH_VDD_VADJ
- wire segments 76 -> 84
- no-connect marks 0 -> 2
Changed lines of the file:
@@
 $Descr A4 11693 8268
 encoding utf-8
-Sheet 4 10
+Sheet 4 46
 Title ""
 Date ""
@@
 AR Path="/61943BD3" Ref="IC?"  Part="1"
 AR Path="/6193F705/61943BD3" Ref="IC?"  Part="1"
+AR Path="/6191D89C/6191EB86/61943BD3" Ref="IC?"  Part="1"
+AR Path="/6191D89C/6191F185/61943BD3" Ref="IC?"  Part="1"
+AR Path="/6191D89C/6192061E/61943BD3" Ref="IC?"  Part="1"
+AR Path="/6191D89C/61920A25/61943BD3" Ref="IC?"  Part="1"
+AR Path="/6191D89C/61933123/61943BD3" Ref="IC?"  Part="1"
+AR Path="/6191D89C/61935424/61943BD3" Ref="IC?"  Part="1"
 F 0 "IC?" H 7750 3700 50  0000 C CNN
 F 1 "PI3WVR628XBEX" H 7750 3550 50  0000 C CNN
@@
 Wire Wire Line
 	4850 5300 7050 5300
-Text HLabel 9200 2650 2    50   Input ~ 0
+Text HLabel 9200 2650 2    50   Output ~ 0
 JETSON_MIPI_CLK_P
-Text HLabel 9200 2750 2    50   Input ~ 0
+Text HLabel 9200 2750 2    50   Output ~ 0
 JETSON_MIPI_CLK_N
-Text HLabel 9200 2850 2    50   Input ~ 0
+Text HLabel 9200 2850 2    50   Output ~ 0
 JETSON_MIPI_D0_P
-Text HLabel 9200 3050 2    50   Input ~ 0
+Text HLabel 9200 3050 2    50   Output ~ 0
 JETSON_MIPI_D1_P
-Text HLabel 9200 3150 2    50   Input ~ 0
+Text HLabel 9200 3150 2    50   Output ~ 0
 JETSON_MIPI_D1_N
-Text HLabel 9200 2950 2    50   Input ~ 0
+Text HLabel 9200 2950 2    50   Output ~ 0
 JETSON_MIPI_D0_N
 Wire Wire Line
@@
 U 1 1 6197263A
 P 8500 3650
+AR Path="/6193F705/6197263A" Ref="#PWR?"  Part="1"
+AR Path="/6191D89C/6191EB86/6197263A" Ref="#PWR?"  Part="1"
+AR Path="/6191D89C/6191F185/6197263A" Ref="#PWR?"  Part="1"
+AR Path="/6191D89C/6192061E/6197263A" Ref="#PWR?"  Part="1"
+AR Path="/6191D89C/61920A25/6197263A" Ref="#PWR?"  Part="1"
+AR Path="/6191D89C/61933123/6197263A" Ref="#PWR?"  Part="1"
+AR Path="/6191D89C/61935424/6197263A" Ref="#PWR?"  Part="1"
 F 0 "#PWR?" H 8500 3400 50  0001 C CNN
 F 1 "Earth" H 8500 3500 50  0001 C CNN
@@
 Wire Wire Line
 	1900 4800 2850 4800
+NoConn ~ 8350 3300
+NoConn ~ 8350 3400
+Wire Wire Line
+	8350 2400 8700 2400
+$Comp
+L Device:R R?
+U 1 1 61907CF0
+P 8850 2400
+AR Path="/595357E2/59539608/61907CF0" Ref="R?"  Part="1"
+AR Path="/595357E2/5953B622/61907CF0" Ref="R?"  Part="1"
+AR Path="/595357E2/5953B846/61907CF0" Ref="R?"  Part="1"
+AR Path="/595357E2/5953BBD4/61907CF0" Ref="R?"  Part="1"
+AR Path="/595357E2/5953D01F/61907CF0" Ref="R?"  Part="1"
+AR Path="/61907CF0" Ref="R?"  Part="1"
+AR Path="/6193F705/61946DF5/61907CF0" Ref="R?"  Part="1"
+AR Path="/6193F705/61958A60/61907CF0" Ref="R?"  Part="1"
+AR Path="/6193F705/61958BD7/61907CF0" Ref="R?"  Part="1"
+AR Path="/6193F705/61958D9F/61907CF0" Ref="R?"  Part="1"
+AR Path="/6193F705/61958F85/61907CF0" Ref="R?"  Part="1"
+AR Path="/6193F705/61959195/61907CF0" Ref="R?"  Part="1"
+AR Path="/6193F705/61907CF0" Ref="R?"  Part="1"
+AR Path="/6191D89C/6191EB86/61907CF0" Ref="R?"  Part="1"
+AR Path="/6191D89C/6191F185/61907CF0" Ref="R?"  Part="1"
+AR Path="/6191D89C/6192061E/61907CF0" Ref="R?"  Part="1"
+AR Path="/6191D89C/61920A25/61907CF0" Ref="R?"  Part="1"
+AR Path="/6191D89C/61933123/61907CF0" Ref="R?"  Part="1"
+AR Path="/6191D89C/61935424/61907CF0" Ref="R?"  Part="1"
+F 0 "R?" V 8930 2400 50  0000 C CNN
+F 1 "4.7K" V 8850 2400 50  0000 C CNN
+F 2 "Resistors_SMD:R_0805" V 8780 2400 50  0001 C CNN
+F 3 "" H 8850 2400 50  0001 C CNN
+F 4 "1%" V 8850 2400 60  0001 C CNN "Tolerance"
+F 5 "1/8W" V 8850 2400 60  0001 C CNN "Power"
+F 6 "RC0805FR-07220RL" V 8850 2400 60  0001 C CNN "Part Number"
+	1    8850 2400
+	0    1    1    0
+$EndComp
+$Comp
+L FMC_MIPI_v2:Earth #PWR?
+U 1 1 6190C0AE
+P 9600 2100
+AR Path="/6193F705/6190C0AE" Ref="#PWR?"  Part="1"
+AR Path="/6191D89C/6191EB86/6190C0AE" Ref="#PWR?"  Part="1"
+AR Path="/6191D89C/6191F185/6190C0AE" Ref="#PWR?"  Part="1"
+AR Path="/6191D89C/6192061E/6190C0AE" Ref="#PWR?"  Part="1"
+AR Path="/6191D89C/61920A25/6190C0AE" Ref="#PWR?"  Part="1"
+AR Path="/6191D89C/61933123/6190C0AE" Ref="#PWR?"  Part="1"
+AR Path="/6191D89C/61935424/6190C0AE" Ref="#PWR?"  Part="1"
+F 0 "#PWR?" H 9600 1850 50  0001 C CNN
+F 1 "Earth" H 9600 1950 50  0001 C CNN
+F 2 "" H 9600 2100 50  0001 C CNN
+F 3 "~" H 9600 2100 50  0001 C CNN
+	1    9600 2100
+	1    0    0    -1
+$EndComp
+Wire Wire Line
+	9000 2400 9000 2000
+Wire Wire Line
+	9000 2000 9600 2000
+Wire Wire Line
+	9600 2000 9600 2100
+Wire Wire Line
+	8350 2500 9200 2500
+Text HLabel 9200 2500 2    50   Input ~ 0
+SWITCH_SEL_VADJ
+Wire Wire Line
+	8350 2300 8600 2300
+Wire Wire Line
+	8600 2300 8600 1800
+Wire Wire Line
+	8600 1800 9200 1800
+Text HLabel 9200 1800 2    50   Input ~ 0
+SWITCH_VDD_VADJ
 $EndSCHEMATC
