File: Level_shift_and_switch.sch (KiCad schematic (older format))
At the start: 5 parts, among them U1 SN74AVCH16T245_DGV_48

Commit message: good, added re-driver
Parts:
- added Q1: BSS138, Package_TO_SOT_SMD:SOT-23, symbol Transistor_FET:BSS138
- added R1, R2: 0, Resistors_SMD:R_0805, symbol Device:R
- added U2: TS3DDR3812_RUA_42, FMC_MIPI_v2_sym:TS3DDR3812RUAR, symbol FMC_MIPI_v2:TS3DDR3812_RUA_42
Connections:
- net BOT_VADJ_LP_CLK_N: now also U1.8 (1B5); no longer U1.22 (2B7)
- net BOT_VADJ_LP_CLK_P: now also U1.9 (1B6); no longer U1.23 (2B8)
- net BOT_VADJ_LP_D0_N: now also U1.5 (1B3); no longer U1.19 (2B5)
- net BOT_VADJ_LP_D0_P: now also U1.6 (1B4); no longer U1.20 (2B6)
- net BOT_VADJ_LP_D1_N: now also U1.2 (1B1); no longer U1.16 (2B3)
- net BOT_VADJ_LP_D1_P: now also U1.3 (1B2); no longer U1.17 (2B4)
- net Earth: now also U2.43 (EPAD), U2.V (GND), U2.V_1 (GND), U2.V_10 (GND), U2.V_11 (GND), U2.V_12 (GND), U2.V_13 (GND), U2.V_14 (GND), U2.V_15 (GND), U2.V_16 (GND), U2.V_17 (GND), U2.V_2 (GND), U2.V_3 (GND), U2.V_4 (GND), U2.V_5 (GND), U2.V_6 (GND), U2.V_7 (GND), U2.V_8 (GND), U2.V_9 (GND)
- net TOP_VADJ_LP_CLK_N: now also U1.16 (2B3); no longer U1.8 (1B5)
- net TOP_VADJ_LP_CLK_P: now also U1.17 (2B4); no longer U1.9 (1B6)
- net TOP_VADJ_LP_D0_N: now also U1.19 (2B5); no longer U1.5 (1B3)
- net TOP_VADJ_LP_D0_P: now also U1.20 (2B6); no longer U1.6 (1B4)
- net TOP_VADJ_LP_D1_N: now also U1.22 (2B7); no longer U1.2 (1B1)
- net TOP_VADJ_LP_D1_P: now also U1.23 (2B8); no longer U1.3 (1B2)
- net SWITCH_VDD_VADJ renamed VDD_VADJ
- net sheet61A8362B/LP_CLK_N renamed BOT_1P2_LP_CLK_N
- net BOT_1P2_LP_CLK_N: now also U2.33 (C4)
- net sheet61A8362B/LP_CLK_P renamed BOT_1P2_LP_CLK_P
- net BOT_1P2_LP_CLK_P: now also U2.31 (C5)
- net sheet61A8362B/LP_D0_N renamed BOT_1P2_LP_D0_N
- net BOT_1P2_LP_D0_N: now also U2.37 (C2)
- net sheet61A8362B/LP_D0_P renamed BOT_1P2_LP_D0_P
- net BOT_1P2_LP_D0_P: now also U2.35 (C3)
- net sheet61A8362B/LP_D1_N renamed BOT_1P2_LP_D1_N
- net BOT_1P2_LP_D1_N: now also U2.42 (C0)
- net sheet61A8362B/LP_D1_P renamed BOT_1P2_LP_D1_P
- net BOT_1P2_LP_D1_P: now also U2.40 (C1)
- net sheet61A8362C/LP_CLK_N renamed TOP_1P2_LP_D1_N
- net TOP_1P2_LP_D1_N: now also U2.20 (C10)
- net sheet61A8362C/LP_CLK_P renamed TOP_1P2_LP_D1_P
- net TOP_1P2_LP_D1_P: now also U2.18 (C11)
- net sheet61A8362C/LP_D0_N renamed TOP_1P2_LP_D0_N
- net TOP_1P2_LP_D0_N: now also U2.24 (C8)
- net sheet61A8362C/LP_D0_P renamed TOP_1P2_LP_D0_P
- net TOP_1P2_LP_D0_P: now also U2.22 (C9)
- net sheet61A8362C/LP_D1_N renamed TOP_1P2_LP_CLK_N
- net TOP_1P2_LP_CLK_N: now also U2.28 (C6)
- net sheet61A8362C/LP_D1_P renamed TOP_1P2_LP_CLK_P
- net TOP_1P2_LP_CLK_P: now also U2.26 (C7)
- new net: R1.1, U2.10 (SEL2), U2.9 (SEL1)
- new net: R2.1, U2.8 (EN)
- new net BOT_JT_MIPI_CLK_N: U2.6 (A4)
- new net BOT_JT_MIPI_CLK_P: U2.7 (A5)
- new net BOT_JT_MIPI_D0_N: U2.4 (A2)
- new net BOT_JT_MIPI_D0_P: U2.5 (A3)
- new net BOT_JT_MIPI_D1_N: U2.2 (A0)
- new net BOT_JT_MIPI_D1_P: U2.3 (A1)
- new net BOT_RDR_HS_CLK_N: U2.34 (B4)
- new net BOT_RDR_HS_CLK_P: U2.32 (B5)
- new net BOT_RDR_HS_D0_N: U2.38 (B2)
- new net BOT_RDR_HS_D0_P: U2.36 (B3)
- new net BOT_RDR_HS_D1_N: U2.41 (B0)
- new net BOT_RDR_HS_D1_P: U2.39 (B1)
- new net SWITCH_HS_0_LP_1_3V3: R1.2
- new net TOP_JT_MIPI_CLK_N: U2.11 (A6)
- new net TOP_JT_MIPI_CLK_P: U2.12 (A7)
- new net TOP_JT_MIPI_D0_N: U2.13 (A8)
- new net TOP_JT_MIPI_D0_P: U2.14 (A9)
- new net TOP_JT_MIPI_D1_N: U2.15 (A10)
- new net TOP_JT_MIPI_D1_P: U2.16 (A11)
- new net TOP_RDR_HS_CLK_N: U2.29 (B6)
- new net TOP_RDR_HS_CLK_P: U2.27 (B7)
- new net TOP_RDR_HS_D0_N: U2.25 (B8)
- new net TOP_RDR_HS_D0_P: U2.23 (B9)
- new net TOP_RDR_HS_D1_N: U2.21 (B10)
- new net TOP_RDR_HS_D1_P: U2.19 (B11)
- new net VOLT_3P3: R2.2, U2.1 (VCC), U2.17 (VCC), U2.30 (VCC)
Other:
- note added: "CML/LVDS Redriver\n"
- note added: "Check CBTV24DD12 and TS3DDR4000!!!\n"
- note added: "High speed switch"
- note added: "Level shifting"
- note added: "TODO: Not mandatory, but good idea to add level shifters to SWITCH_HS_0_LP_1_3V3\nhttp://cdn.sparkfun.com/datasheets/BreakoutBoards/Logic_Level_Bidirectional.pdf\nTest it!!"

Commit message: good, before reducing
Parts:
- removed Q1: BSS138, Package_TO_SOT_SMD:SOT-23, symbol Transistor_FET:BSS138
- added C17, C18, C19: 0.1uF, Capacitors_SMD:C_0402, symbol FMC_MIPI_v2:C
- added U5: SN74LV1T34DBV, TO_SOT_Packages_SMD:SOT-23-5, symbol Logic_LevelTranslator:SN74LV1T34DBV
Connections:
- net Earth: now also C17.2, C18.2, C19.2, U5.3 (GND)
- net SWITCH_HS_0_LP_1_3V3: now also U5.4 (Y)
- net VOLT_3P3: now also C17.1, C18.1, C19.1, U5.5 (VCC)
- new net SWITCH_HS_0_LP_1_VADJ: U5.2 (A)
Other:
- note added: "Decoupling for TS3DDR3812_RUA_42"
- note added: "Switch SEL1,2 level shift to 3p3 volt"
- note removed: "TODO: Not mandatory, but good idea to add level shifters to SWITCH_HS_0_LP_1_3V3\nhttp://cdn.sparkfun.com/datasheets/BreakoutBoards/Logic_Level_Bidirectional.pdf\nTest it!!"
- moved on the sheet: C1, C2, C3, C4, R1, R2, U1, U2
