File: LVDS_2_SLVS_experimental.sch (KiCad schematic (older format))
At the start: 6 parts

Commit message: rev 2022
Parts:
- removed R12, R13: 220, Resistors_SMD:R_0603, symbol Device:R
- removed R14, R15: 47, Resistors_SMD:R_0603, symbol Device:R
- added R30, R31: 220, Resistors_SMD:R_0603, symbol Device:R
- added R32, R33: 47, Resistors_SMD:R_0603, symbol Device:R
Connections:
- net LVDS_IN_N: now also R31.2, R33.2
- net LVDS_IN_P: now also R30.1, R32.2
- net SLVS_OUT_N: now also R33.1
- net SLVS_OUT_P: now also R32.1
- net VOLT_2P5: now also R30.2, R31.1
