File: Level_shift_and_switch_single.sch (KiCad schematic (older format))
At the start: 13 parts, among them U1 SN74AVCH16T245_DGV_48, U2 TS3DDR3812_RUA_42, U3 SN74LV1T34DBV

Commit message: rev 2022
Connections:
- wire segments 168 -> 169
