File: LVDS_to_Jetson_lines.sch (KiCad schematic (older format))
At the start: 15 parts, among them U5 TS3DDR3812_RUA_42, U6 TS3DDR3812_RUA_42, U8 SN74AVCH16T245_DGV_48

Commit message: minor changes
Connections:
- net labels added: FMC_LP_CSI_C_CLK_N, FMC_LP_CSI_C_CLK_P, FMC_LP_CSI_C_D0_N, FMC_LP_CSI_C_D0_P, FMC_LP_CSI_C_D1_N, FMC_LP_CSI_C_D1_P, FMC_LP_CSI_D_CLK_N, FMC_LP_CSI_D_CLK_P, FMC_LP_CSI_D_D0_N, FMC_LP_CSI_D_D0_P, FMC_LP_CSI_D_D1_N, FMC_LP_CSI_D_D1_P
- net labels removed: fdmkls_TOP_VADJ_LP_CLK_N, fdmkls_TOP_VADJ_LP_CLK_P, fdmkls_TOP_VADJ_LP_D0_N, fdmkls_TOP_VADJ_LP_D0_P, fdmkls_TOP_VADJ_LP_D1_N, fdmkls_TOP_VADJ_LP_D1_P
Changed lines of the file:
@@
 Text GLabel 14650 3350 2    50   Output ~ 0
 CSI_D_D0_N
-Text GLabel 14750 6700 2    50   Output ~ 0
+Text GLabel 14750 7100 2    50   Output ~ 0
 CSI_D_CLK_P
-Text GLabel 14750 6600 2    50   Output ~ 0
+Text GLabel 14750 7000 2    50   Output ~ 0
 CSI_D_CLK_N
 Text GLabel 14650 3250 2    50   Output ~ 0
@@
 Wire Wire Line
 	14450 7100 14750 7100
-Text GLabel 14750 7000 2    50   Output ~ 0
+Text GLabel 14750 6600 2    50   Output ~ 0
 CSI_C_CLK_N
-Text GLabel 14750 7100 2    50   Output ~ 0
+Text GLabel 14750 6700 2    50   Output ~ 0
 CSI_C_CLK_P
 Wire Wire Line
@@
 Wire Wire Line
 	6600 8800 6600 8900
-$Comp
-L FMC_MIPI_v2:Earth #PWR?
-U 1 1 63571F8A
-P 7050 8850
-AR Path="/6193F705/63571F8A" Ref="#PWR?"  Part="1"
-AR Path="/6191D89C/6191EB86/63571F8A" Ref="#PWR?"  Part="1"
-AR Path="/6191D89C/6191F185/63571F8A" Ref="#PWR?"  Part="1"
-AR Path="/6191D89C/6192061E/63571F8A" Ref="#PWR?"  Part="1"
-AR Path="/6191D89C/61920A25/63571F8A" Ref="#PWR?"  Part="1"
-AR Path="/6191D89C/61933123/63571F8A" Ref="#PWR?"  Part="1"
-AR Path="/6191D89C/61935424/63571F8A" Ref="#PWR?"  Part="1"
-AR Path="/6191D89C/63571F8A" Ref="#PWR0107"  Part="1"
-AR Path="/6191D89C/61A814B9/63571F8A" Ref="#PWR?"  Part="1"
-AR Path="/6191D89C/61A38142/63571F8A" Ref="#PWR?"  Part="1"
-AR Path="/6191D89C/61A4C646/63571F8A" Ref="#PWR?"  Part="1"
-AR Path="/6191D89C/62016C67/63571F8A" Ref="#PWR?"  Part="1"
-F 0 "#PWR0107" H 7050 8600 50  0001 C CNN
-F 1 "Earth" H 7050 8700 50  0001 C CNN
-F 2 "" H 7050 8850 50  0001 C CNN
-F 3 "~" H 7050 8850 50  0001 C CNN
-	1    7050 8850
-	1    0    0    -1
-$EndComp
 Wire Wire Line
 	7050 8700 7050 8850
@@
 Wire Wire Line
 	3900 8800 3900 8900
-Wire Wire Line
-	3150 9400 4050 9400
-Wire Wire Line
-	4050 9500 3150 9500
-Wire Wire Line
-	3150 9700 4050 9700
-Wire Wire Line
-	4050 9800 3150 9800
 $Comp
 L FMC_MIPI_v2:C C?
@@
 Text Notes 4700 7100 0    118  ~ 0
 Level shifting
-Wire Wire Line
-	6450 9400 6950 9400
-Wire Wire Line
-	6950 9400 6950 9300
-Text HLabel 3400 8300 0    50   Input ~ 0
-fdmkls_TOP_VADJ_LP_D1_N
-Text HLabel 3200 8600 0    50   Input ~ 0
-fdmkls_TOP_VADJ_LP_D1_P
 Connection ~ 6700 8200
 $Comp
@@
 Text Label 7500 7450 0    50   ~ 10
 VOLT_1P2
-Wire Wire Line
-	7050 9500 7050 9400
-Wire Wire Line
-	6450 9700 7200 9700
-Wire Wire Line
-	7200 9700 7200 9500
-Wire Wire Line
-	6450 9800 7300 9800
-Wire Wire Line
-	7300 9800 7300 9600
-Wire Wire Line
-	3400 8300 4050 8300
 Wire Wire Line
 	6600 8700 7050 8700
@@
 	1    0    0    -1
 $EndComp
-$Comp
-L FMC_MIPI_v2:Earth #PWR?
-U 1 1 63572036
-P 7050 8850
-AR Path="/6193F705/63572036" Ref="#PWR?"  Part="1"
-AR Path="/6191D89C/6191EB86/63572036" Ref="#PWR?"  Part="1"
-AR Path="/6191D89C/6191F185/63572036" Ref="#PWR?"  Part="1"
-AR Path="/6191D89C/6192061E/63572036" Ref="#PWR?"  Part="1"
-AR Path="/6191D89C/61920A25/63572036" Ref="#PWR?"  Part="1"
-AR Path="/6191D89C/61933123/63572036" Ref="#PWR?"  Part="1"
-AR Path="/6191D89C/61935424/63572036" Ref="#PWR?"  Part="1"
-AR Path="/6191D89C/63572036" Ref="#PWR0111"  Part="1"
-AR Path="/6191D89C/61A814B9/63572036" Ref="#PWR?"  Part="1"
-AR Path="/6191D89C/61A38142/63572036" Ref="#PWR?"  Part="1"
-AR Path="/6191D89C/61A4C646/63572036" Ref="#PWR?"  Part="1"
-AR Path="/6191D89C/62016C67/63572036" Ref="#PWR?"  Part="1"
-F 0 "#PWR0111" H 7050 8600 50  0001 C CNN
-F 1 "Earth" H 7050 8700 50  0001 C CNN
-F 2 "" H 7050 8850 50  0001 C CNN
-F 3 "~" H 7050 8850 50  0001 C CNN
-	1    7050 8850
-	1    0    0    -1
-$EndComp
-$Comp
-L FMC_MIPI_v2:Earth #PWR?
-U 1 1 6357203D
-P 3250 8750
-AR Path="/6193F705/6357203D" Ref="#PWR?"  Part="1"
-AR Path="/6191D89C/6191EB86/6357203D" Ref="#PWR?"  Part="1"
-AR Path="/6191D89C/6191F185/6357203D" Ref="#PWR?"  Part="1"
-AR Path="/6191D89C/6192061E/6357203D" Ref="#PWR?"  Part="1"
-AR Path="/6191D89C/61920A25/6357203D" Ref="#PWR?"  Part="1"
-AR Path="/6191D89C/61933123/6357203D" Ref="#PWR?"  Part="1"
-AR Path="/6191D89C/61935424/6357203D" Ref="#PWR?"  Part="1"
-AR Path="/6191D89C/6357203D" Ref="#PWR0112"  Part="1"
-AR Path="/6191D89C/61A814B9/6357203D" Ref="#PWR?"  Part="1"
-AR Path="/6191D89C/61A38142/6357203D" Ref="#PWR?"  Part="1"
-AR Path="/6191D89C/61A4C646/6357203D" Ref="#PWR?"  Part="1"
-AR Path="/6191D89C/62016C67/6357203D" Ref="#PWR?"  Part="1"
-F 0 "#PWR0112" H 3250 8500 50  0001 C CNN
-F 1 "Earth" H 3250 8600 50  0001 C CNN
-F 2 "" H 3250 8750 50  0001 C CNN
-F 3 "~" H 3250 8750 50  0001 C CNN
-	1    3250 8750
-	1    0    0    -1
-$EndComp
-Text HLabel 3150 9400 0    50   Input ~ 0
-fdmkls_TOP_VADJ_LP_CLK_N
-Text HLabel 3150 9500 0    50   Input ~ 0
-fdmkls_TOP_VADJ_LP_CLK_P
-Text HLabel 3150 9700 0    50   Input ~ 0
-fdmkls_TOP_VADJ_LP_D0_N
-Text HLabel 3150 9800 0    50   Input ~ 0
-fdmkls_TOP_VADJ_LP_D0_P
-Connection ~ 3250 8750
-Connection ~ 7050 8850
 Text Notes 12750 2200 0    50   ~ 0
 LP/HS switch data lanes
@@
 Wire Wire Line
 	12050 7100 11400 7100
+Text Label 11300 8400 0    50   ~ 0
+LP_CSI_D_CLK_N
+Text Label 11300 8500 0    50   ~ 0
+LP_CSI_D_CLK_P
 Text Label 11300 8000 0    50   ~ 0
-LP_CSI_D_CLK_N
+LP_CSI_C_CLK_N
 Text Label 11300 8100 0    50   ~ 0
-LP_CSI_D_CLK_P
-Text Label 11300 8400 0    50   ~ 0
-LP_CSI_C_CLK_N
-Text Label 11300 8500 0    50   ~ 0
 LP_CSI_C_CLK_P
 Wire Wire Line
@@
 Text Label 7900 8000 2    50   ~ 0
 LP_CSI_C_CLK_N
-Text Label 7900 8400 2    50   ~ 0
+Text Label 7850 8400 2    50   ~ 0
 LP_CSI_C_D1_P
-Text Label 7900 8300 2    50   ~ 0
+Text Label 7850 8300 2    50   ~ 0
 LP_CSI_C_D1_N
 Text Label 7900 9100 2    50   ~ 0
@@
 Text Label 7900 9200 2    50   ~ 0
 LP_CSI_C_D0_P
-Text Label 7950 9300 2    50   ~ 0
-LP_CSI_D_D1_N
-Text Label 7950 9400 2    50   ~ 0
-LP_CSI_D_D1_P
-Text Label 7950 9600 2    50   ~ 0
-LP_CSI_D_D0_P
-Text Label 7950 9500 2    50   ~ 0
-LP_CSI_D_D0_N
 Text Notes 7850 8800 2    50   ~ 0
 LP lanes
@@
 	6450 9200 7900 9200
 Wire Wire Line
-	6450 8300 7900 8300
-Wire Wire Line
-	6450 8400 7900 8400
+	6450 8300 7850 8300
+Wire Wire Line
+	6450 8400 7850 8400
 Wire Wire Line
 	6450 8000 7900 8000
@@
 Wire Wire Line
 	6600 8600 6600 8700
-Wire Wire Line
-	3200 8600 3400 8600
 Wire Wire Line
 	6450 7700 7900 7700
@@
 	1    0    0    -1
 $EndComp
-Wire Wire Line
-	6450 9500 7050 9500
 Text Label 7900 7700 2    50   ~ 0
 LP_CSI_D_CLK_N
 Text Label 7900 7800 2    50   ~ 0
 LP_CSI_D_CLK_P
-Wire Wire Line
-	7950 9600 7300 9600
-Wire Wire Line
-	7950 9500 7200 9500
-Wire Wire Line
-	7050 9400 7950 9400
-Wire Wire Line
-	6950 9300 7950 9300
 Text Notes 4700 6650 0    50   ~ 0
 Note: LP signal are single ended!! No need to treat them as diffrential,\n+ they are low speed, so SI is not an issue.\nPlacing it at the bottom layer for now.
@@
 Wire Wire Line
 	12050 3150 11450 3150
+Text Label 11400 7000 0    50   ~ 0
+HS_CSI_D_CLK_N
+Text Label 11400 7100 0    50   ~ 0
+HS_CSI_D_CLK_P
 Text Label 11400 6600 0    50   ~ 0
-HS_CSI_D_CLK_N
+HS_CSI_C_CLK_N
 Text Label 11400 6700 0    50   ~ 0
-HS_CSI_D_CLK_P
-Text Label 11400 7000 0    50   ~ 0
-HS_CSI_C_CLK_N
-Text Label 11400 7100 0    50   ~ 0
 HS_CSI_C_CLK_P
 Text Label 6750 1800 0    50   ~ 10
@@
 Text Label 6400 4100 0    50   ~ 0
 FMC_HS_CSI_D_D0_P
-Text Label 6400 4700 0    50   ~ 0
-FMC_HS_CSI_D_CLK_N
 Text Label 6400 4800 0    50   ~ 0
 FMC_HS_CSI_D_CLK_P
@@
 Wire Wire Line
 	7300 5450 6400 5450
+Text Label 6400 4700 0    50   ~ 0
+FMC_HS_CSI_D_CLK_N
+Text Label 3200 8100 2    50   ~ 0
+FMC_LP_CSI_C_CLK_P
+Text Label 3200 8000 2    50   ~ 0
+FMC_LP_CSI_C_CLK_N
+Text Label 3200 8400 2    50   ~ 0
+FMC_LP_CSI_C_D1_P
+Text Label 3200 8300 2    50   ~ 0
+FMC_LP_CSI_C_D1_N
+Text Label 3200 9100 2    50   ~ 0
+FMC_LP_CSI_C_D0_N
+Text Label 3200 9200 2    50   ~ 0
+FMC_LP_CSI_C_D0_P
+Text Label 3200 9400 2    50   ~ 0
+FMC_LP_CSI_D_D1_N
+Text Label 3200 9500 2    50   ~ 0
+FMC_LP_CSI_D_D1_P
+Text Label 3200 9800 2    50   ~ 0
+FMC_LP_CSI_D_D0_P
+Text Label 3200 9700 2    50   ~ 0
+FMC_LP_CSI_D_D0_N
+Text Notes 2750 8600 2    50   ~ 0
+LP lanes
+Text Label 3200 7700 2    50   ~ 0
+FMC_LP_CSI_D_CLK_N
+Text Label 3200 7800 2    50   ~ 0
+FMC_LP_CSI_D_CLK_P
+Wire Wire Line
+	3200 7700 4050 7700
+Wire Wire Line
+	4050 7800 3200 7800
+Wire Wire Line
+	3200 8000 4050 8000
+Wire Wire Line
+	4050 8100 3200 8100
+Wire Wire Line
+	3200 8300 4050 8300
+Wire Wire Line
+	4050 8400 3200 8400
+Wire Wire Line
+	3200 9100 4050 9100
+Wire Wire Line
+	4050 9200 3200 9200
+Text Label 7900 9700 2    50   ~ 0
+LP_CSI_D_D0_N
+Text Label 7900 9800 2    50   ~ 0
+LP_CSI_D_D0_P
+Text Label 7900 9500 2    50   ~ 0
+LP_CSI_D_D1_P
+Text Label 7900 9400 2    50   ~ 0
+LP_CSI_D_D1_N
+Wire Wire Line
+	6450 9400 7900 9400
+Wire Wire Line
+	6450 9500 7900 9500
+Wire Wire Line
+	6450 9700 7900 9700
+Wire Wire Line
+	6450 9800 7900 9800
+$Comp
+L FMC_MIPI_v2:Earth #PWR?
+U 1 1 63572036
+P 7050 8850
+AR Path="/6193F705/63572036" Ref="#PWR?"  Part="1"
+AR Path="/6191D89C/6191EB86/63572036" Ref="#PWR?"  Part="1"
+AR Path="/6191D89C/6191F185/63572036" Ref="#PWR?"  Part="1"
+AR Path="/6191D89C/6192061E/63572036" Ref="#PWR?"  Part="1"
+AR Path="/6191D89C/61920A25/63572036" Ref="#PWR?"  Part="1"
+AR Path="/6191D89C/61933123/63572036" Ref="#PWR?"  Part="1"
+AR Path="/6191D89C/61935424/63572036" Ref="#PWR?"  Part="1"
+AR Path="/6191D89C/63572036" Ref="#PWR0111"  Part="1"
+AR Path="/6191D89C/61A814B9/63572036" Ref="#PWR?"  Part="1"
+AR Path="/6191D89C/61A38142/63572036" Ref="#PWR?"  Part="1"
+AR Path="/6191D89C/61A4C646/63572036" Ref="#PWR?"  Part="1"
+AR Path="/6191D89C/62016C67/63572036" Ref="#PWR?"  Part="1"
+F 0 "#PWR0111" H 7050 8600 50  0001 C CNN
+F 1 "Earth" H 7050 8700 50  0001 C CNN
+F 2 "" H 7050 8850 50  0001 C CNN
+F 3 "~" H 7050 8850 50  0001 C CNN
+	1    7050 8850
+	1    0    0    -1
+$EndComp
+Wire Wire Line
+	4050 8600 3900 8600
+Wire Wire Line
+	3900 8600 3900 8700
+Wire Wire Line
+	3200 9700 4050 9700
+Wire Wire Line
+	3200 9800 4050 9800
+Wire Wire Line
+	3200 9400 4050 9400
+Wire Wire Line
+	3200 9500 4050 9500
 $EndSCHEMATC

Commit message: good, before completely removing redriver part
Parts:
- added R75: 0, Resistors_SMD:R_0805, symbol Device:R
- added U7: SN74LV1T34DBV, TO_SOT_Packages_SMD:SOT-23-5, symbol Logic_LevelTranslator:SN74LV1T34DBV
Connections:
- net labels added: SWITCH_DATA_LANES_3V3, SWITCH_DATA_LANES_VADJ, SWITCH_U5
- wire segments 250 -> 260
Other:
- note added: "Switch SEL1,2 level shift to 3p3 volt"
- moved on the sheet: C18, C19, C20

Commit message: fixed 3.3 volt level shifter
Parts:
- removed U7: SN74LV1T34DBV, TO_SOT_Packages_SMD:SOT-23-5, symbol Logic_LevelTranslator:SN74LV1T34DBV
- added C1, C2: 0.1uF, Capacitors_SMD:C_0402, symbol FMC_MIPI_v2:C
- added R1, R2: 0, Resistors_SMD:R_0805, symbol Device:R
- added U2: SN74AVC2T45DCUR, FMC_MIPI_v2_sym:SN74AVC2T45DCUR, symbol FMC_MIPI_v2:SN74AVC2T45DCUR
Connections:
- net labels added: DIR, FMC_SWITCH_CLOCK_LANES_VADJ, FMC_SWITCH_DATA_LANES_VADJ, SWITCH_CLOCK_LANES_3V3, SWITCH_U6
- net labels removed: SWITCH_DATA_LANES_VADJ, SWITCH_HS_LV_CAM_C
- wire segments 260 -> 269
Other:
- note added: "Decoupling capacitors U2"
- note added: "Level shifting VADJ to MIPI LP VOLT_1P2"
- note added: "NOTE: use CSI A and CSI B from the same IC, since they can form 4 lane configuration\n"
- note added: "Switches U5 and U6, SEL1,2 level shift from VADJ to 3p3 volt"
- note added: "TODO: make LP lanes split from a single FMC source!!\nClock LP lanes as well!!\n Split goes here!!"
- note removed: "BUG: use CSI A and CSI B from the same IC, since they can form 4 lane configuration\n"
- note removed: "Level shifting"
- note removed: "Switch SEL1,2 level shift to 3p3 volt"
