File: FMC_MIPI_v2.kicad_pcb (KiCad board)
At the start: 6 copper layers, 69 x 112 mm, 5 parts, among them IC1 HD3SS3411TRWARQ1, IC2 HD3SS3411TRWARQ1, IC3 PI3WVR628XBEX, J1 ASP-134488-01, J2 QTH-060-01-L-D-A

Commit message: Good, before replacing the swithches to TI ones
Parts:
- added C1: 0.1uF, Capacitors_SMD:C_0402, B.Cu at (-8.00, 70.8)
- added C10: 0.1uF, Capacitors_SMD:C_0402, F.Cu at (-117.8, -65.0)
- added C11: 0.1uF, Capacitors_SMD:C_0402, F.Cu at (-116.5, -46.9)
- added C12: 0.1uF, Capacitors_SMD:C_0402, F.Cu at (-116.5, -44.8)
- added C13: 0.1uF, Capacitors_SMD:C_0402, F.Cu at (-92.2, -42.7)
- added C14: 0.01uF, Capacitors_SMD:C_0402, F.Cu at (-95.2, -42.7)
- added C15: 0.1uF, Capacitors_SMD:C_0402, F.Cu at (-92.4, -61.1)
- added C16: 0.01uF, Capacitors_SMD:C_0402, F.Cu at (-95.4, -61.1)
- added C17: 0.1uF, Capacitors_SMD:C_0402, F.Cu at (-348.1, 105.3)
- added C18: 0.1uF, Capacitors_SMD:C_0402, F.Cu at (-348.1, 107.3)
- added C19: 0.1uF, Capacitors_SMD:C_0402, F.Cu at (-287.6, 172.7)
- added C2: 0.1uF, Capacitors_SMD:C_0402, B.Cu at (-7.90, 75.0)
- added C20: 0.1uF, Capacitors_SMD:C_0402, F.Cu at (-290.7, 172.7)
- added C21: 0.1uF, Capacitors_SMD:C_0402, F.Cu at (-319.8, 135.9)
- added C22: 0.01uF, Capacitors_SMD:C_0402, F.Cu at (-316.7, 135.9)
- added C23: 0.1uF, Capacitors_SMD:C_0402, F.Cu at (-319.8, 127.1)
- added C24: 0.01uF, Capacitors_SMD:C_0402, F.Cu at (-316.7, 127.1)
- added C25: 1uF, Capacitors_SMD:C_0603, F.Cu at (-323.4, 189.6)
- added C26: 1uF, Capacitors_SMD:C_0603, F.Cu at (-331.9, 198.3)
- added C27: 0.1uF, Capacitors_SMD:C_0402, F.Cu at (-327.9, 195.2)
- added C28: 0.1uF, Capacitors_SMD:C_0402, F.Cu at (-323.8, 191.8)
- added C29: 0.1uF, Capacitors_SMD:C_0402, F.Cu at (-327.9, 197.3)
- added C3: 0.1uF, Capacitors_SMD:C_0402, B.Cu at (3.60, 76.2)
- added C30: 0.1uF, Capacitors_SMD:C_0402, F.Cu at (-324.9, 195.2)
- added C4: 0.1uF, Capacitors_SMD:C_0402, B.Cu at (3.50, 70.8)
- added C5: 0.1uF, Capacitors_SMD:C_0402, F.Cu at (5.58, 87.0)
- added C6: 0.01uF, Capacitors_SMD:C_0402, F.Cu at (13.7, 87.2)
- added C7: 0.1uF, Capacitors_SMD:C_0402, F.Cu at (4.08, 65.5)
- added C8: 0.01uF, Capacitors_SMD:C_0402, F.Cu at (9.56, 65.5)
- added C9: 0.1uF, Capacitors_SMD:C_0402, F.Cu at (-120.9, -65.0)
- added IC4: PI3WVR626XEBEX, QFN35P250X250X50-25N, F.Cu at (-107.4, -62.2)
- added IC5: PI3WVR626XEBEX, QFN35P250X250X50-25N, F.Cu at (-330.9, 135.3)
- added IC6: PI3WVR626XEBEX, QFN35P250X250X50-25N, F.Cu at (-330.3, 120.1)
- added R1: 4.7K, Resistors_SMD:R_0805, F.Cu at (9.85, 88.0)
- added R10: 47, Resistors_SMD:R_0805, F.Cu at (-19.9, 83.6)
- added R100: 47, Resistors_SMD:R_0805, F.Cu at (-274.2, 129.0)
- added R101: 9, Resistors_SMD:R_0805, F.Cu at (-274.2, 126.1)
- added R102: 9, Resistors_SMD:R_0805, F.Cu at (-278.3, 129.0)
- added R103: 4.7K, Resistors_SMD:R_0805, F.Cu at (-319.2, 124.6)
- added R104: 220, Resistors_SMD:R_0805, F.Cu at (-295.9, 186.6)
- added R105: 220, Resistors_SMD:R_0805, F.Cu at (-291.7, 183.7)
- added R106: 47, Resistors_SMD:R_0805, F.Cu at (-291.7, 186.6)
- added R107: 47, Resistors_SMD:R_0805, F.Cu at (-295.9, 183.7)
- added R108: 9, Resistors_SMD:R_0805, F.Cu at (-287.6, 183.7)
- added R109: 9, Resistors_SMD:R_0805, F.Cu at (-287.6, 186.6)
- added R11: 47, Resistors_SMD:R_0805, F.Cu at (-19.9, 80.8)
- added R110: 220, Resistors_SMD:R_0805, F.Cu at (-299.1, 136.8)
- added R111: 220, Resistors_SMD:R_0805, F.Cu at (-299.1, 139.6)
- added R112: 47, Resistors_SMD:R_0805, F.Cu at (-295.0, 136.8)
- added R113: 47, Resistors_SMD:R_0805, F.Cu at (-295.0, 139.6)
- added R114: 9, Resistors_SMD:R_0805, F.Cu at (-290.8, 136.8)
- added R115: 9, Resistors_SMD:R_0805, F.Cu at (-290.8, 139.6)
- added R116: 220, Resistors_SMD:R_0805, F.Cu at (-295.0, 126.1)
- added R117: 220, Resistors_SMD:R_0805, F.Cu at (-299.1, 129.0)
- added R118: 47, Resistors_SMD:R_0805, F.Cu at (-299.1, 126.1)
- added R119: 47, Resistors_SMD:R_0805, F.Cu at (-295.0, 129.0)
- added R12: 9, Resistors_SMD:R_0805, F.Cu at (-24.0, 83.6)
- added R120: 9, Resistors_SMD:R_0805, F.Cu at (-290.8, 126.1)
- added R121: 9, Resistors_SMD:R_0805, F.Cu at (-290.8, 129.0)
- added R122: 4.7k, Resistors_SMD:R_0805, F.Cu at (-340.0, 198.4)
- added R123: 4.7k, Resistors_SMD:R_0805, F.Cu at (-331.5, 189.9)
- added R124: 2.2k, Resistors_SMD:R_0805, F.Cu at (-335.9, 198.4)
- added R125: 2.2k, Resistors_SMD:R_0805, F.Cu at (-331.5, 192.8)
- added R126: 4.7k, Resistors_SMD:R_0805, F.Cu at (-327.4, 189.9)
- added R127: 4.7k, Resistors_SMD:R_0805, F.Cu at (-331.5, 195.7)
- added R128: 4.7k, Resistors_SMD:R_0805, F.Cu at (-327.4, 192.8)
- added R13: 9, Resistors_SMD:R_0805, F.Cu at (-24.0, 80.8)
- added R14: 220, Resistors_SMD:R_0805, F.Cu at (-15.7, 95.8)
- added R15: 220, Resistors_SMD:R_0805, F.Cu at (-24.0, 95.8)
- added R16: 47, Resistors_SMD:R_0805, F.Cu at (-24.0, 98.7)
- added R17: 47, Resistors_SMD:R_0805, F.Cu at (-19.8, 95.8)
- added R18: 9, Resistors_SMD:R_0805, F.Cu at (-19.8, 98.7)
- added R19: 9, Resistors_SMD:R_0805, F.Cu at (-15.7, 98.7)
- added R2: 220, Resistors_SMD:R_0805, F.Cu at (-24.1, 90.6)
- added R20: 4.7K, Resistors_SMD:R_0805, F.Cu at (7.06, 63.0)
- added R21: 220, Resistors_SMD:R_0805, F.Cu at (-24.8, 66.7)
- added R22: 220, Resistors_SMD:R_0805, F.Cu at (-24.8, 63.8)
- added R23: 47, Resistors_SMD:R_0805, F.Cu at (-20.6, 63.8)
- added R24: 47, Resistors_SMD:R_0805, F.Cu at (-20.6, 66.7)
- added R25: 9, Resistors_SMD:R_0805, F.Cu at (-16.5, 63.8)
- added R26: 9, Resistors_SMD:R_0805, F.Cu at (-16.5, 66.7)
- added R27: 220, Resistors_SMD:R_0805, F.Cu at (-16.8, 54.7)
- added R28: 220, Resistors_SMD:R_0805, F.Cu at (-21.0, 57.6)
- added R29: 47, Resistors_SMD:R_0805, F.Cu at (-21.0, 54.7)
- added R3: 220, Resistors_SMD:R_0805, F.Cu at (-20.0, 87.7)
- added R30: 47, Resistors_SMD:R_0805, F.Cu at (-25.1, 57.6)
- added R31: 9, Resistors_SMD:R_0805, F.Cu at (-16.8, 57.6)
- added R32: 9, Resistors_SMD:R_0805, F.Cu at (-25.1, 54.7)
- added R33: 220, Resistors_SMD:R_0805, F.Cu at (-24.2, 74.4)
- added R34: 220, Resistors_SMD:R_0805, F.Cu at (-20.0, 71.5)
- added R35: 47, Resistors_SMD:R_0805, F.Cu at (-20.0, 74.4)
- added R36: 47, Resistors_SMD:R_0805, F.Cu at (-15.9, 71.5)
- added R37: 9, Resistors_SMD:R_0805, F.Cu at (-24.2, 71.5)
- added R38: 9, Resistors_SMD:R_0805, F.Cu at (-15.9, 74.4)
- added R39: 4.7K, Resistors_SMD:R_0805, F.Cu at (-94.7, -45.2)
- added R4: 47, Resistors_SMD:R_0805, F.Cu at (-20.0, 90.6)
- added R40: 220, Resistors_SMD:R_0805, F.Cu at (-74.3, -31.8)
- added R41: 220, Resistors_SMD:R_0805, F.Cu at (-74.3, -34.7)
- added R42: 47, Resistors_SMD:R_0805, F.Cu at (-78.4, -31.8)
- added R43: 47, Resistors_SMD:R_0805, F.Cu at (-78.4, -34.7)
- added R44: 9, Resistors_SMD:R_0805, F.Cu at (-82.6, -31.8)
- added R45: 9, Resistors_SMD:R_0805, F.Cu at (-82.6, -34.7)
- added R46: 220, Resistors_SMD:R_0805, F.Cu at (-74.1, -43.7)
- added R47: 220, Resistors_SMD:R_0805, F.Cu at (-74.1, -46.6)
- added R48: 47, Resistors_SMD:R_0805, F.Cu at (-78.3, -43.7)
- added R49: 47, Resistors_SMD:R_0805, F.Cu at (-78.3, -46.6)
- added R5: 47, Resistors_SMD:R_0805, F.Cu at (-15.8, 90.6)
- added R50: 9, Resistors_SMD:R_0805, F.Cu at (-82.4, -46.6)
- added R51: 9, Resistors_SMD:R_0805, F.Cu at (-82.4, -43.7)
- added R52: 220, Resistors_SMD:R_0805, F.Cu at (-82.3, -56.4)
- added R53: 220, Resistors_SMD:R_0805, F.Cu at (-82.3, -53.5)
- added R54: 47, Resistors_SMD:R_0805, F.Cu at (-78.1, -56.4)
- added R55: 47, Resistors_SMD:R_0805, F.Cu at (-78.1, -53.5)
- added R56: 9, Resistors_SMD:R_0805, F.Cu at (-74.0, -56.4)
- added R57: 9, Resistors_SMD:R_0805, F.Cu at (-74.0, -53.5)
- added R58: 4.7K, Resistors_SMD:R_0805, F.Cu at (-94.9, -63.5)
- added R59: 220, Resistors_SMD:R_0805, F.Cu at (-68.9, -66.3)
- added R6: 9, Resistors_SMD:R_0805, F.Cu at (-15.8, 87.7)
- added R60: 220, Resistors_SMD:R_0805, F.Cu at (-68.9, -63.4)
- added R61: 47, Resistors_SMD:R_0805, F.Cu at (-64.7, -66.3)
- added R62: 47, Resistors_SMD:R_0805, F.Cu at (-64.7, -63.4)
- added R63: 9, Resistors_SMD:R_0805, F.Cu at (-60.6, -66.3)
- added R64: 9, Resistors_SMD:R_0805, F.Cu at (-60.6, -63.4)
- added R65: 220, Resistors_SMD:R_0805, F.Cu at (-74.3, -84.7)
- added R66: 220, Resistors_SMD:R_0805, F.Cu at (-82.6, -81.8)
- added R67: 47, Resistors_SMD:R_0805, F.Cu at (-78.4, -84.7)
- added R68: 47, Resistors_SMD:R_0805, F.Cu at (-78.4, -81.8)
- added R69: 9, Resistors_SMD:R_0805, F.Cu at (-82.6, -84.7)
- added R7: 9, Resistors_SMD:R_0805, F.Cu at (-24.1, 87.7)
- added R70: 9, Resistors_SMD:R_0805, F.Cu at (-74.3, -81.8)
- added R71: 220, Resistors_SMD:R_0805, F.Cu at (-60.5, -72.9)
- added R72: 220, Resistors_SMD:R_0805, F.Cu at (-60.5, -75.8)
- added R73: 47, Resistors_SMD:R_0805, F.Cu at (-64.6, -72.9)
- added R74: 47, Resistors_SMD:R_0805, F.Cu at (-64.6, -75.8)
- added R75: 9, Resistors_SMD:R_0805, F.Cu at (-68.8, -72.9)
- added R76: 9, Resistors_SMD:R_0805, F.Cu at (-68.8, -75.8)
- added R77: 220, Resistors_SMD:R_0805, F.Cu at (-294.3, 170.2)
- added R78: 220, Resistors_SMD:R_0805, F.Cu at (-290.1, 167.3)
- added R79: 47, Resistors_SMD:R_0805, F.Cu at (-294.3, 173.1)
- added R8: 220, Resistors_SMD:R_0805, F.Cu at (-15.7, 83.6)
- added R80: 47, Resistors_SMD:R_0805, F.Cu at (-290.1, 170.2)
- added R81: 9, Resistors_SMD:R_0805, F.Cu at (-290.1, 164.4)
- added R82: 9, Resistors_SMD:R_0805, F.Cu at (-294.3, 167.3)
- added R83: 100, Resistors_SMD:R_0805, F.Cu at (-294.3, 164.4)
- added R84: 4.7K, Resistors_SMD:R_0805, F.Cu at (-319.2, 133.5)
- added R85: 220, Resistors_SMD:R_0805, F.Cu at (-308.2, 116.8)
- added R86: 220, Resistors_SMD:R_0805, F.Cu at (-308.2, 113.9)
- added R87: 47, Resistors_SMD:R_0805, F.Cu at (-312.4, 116.8)
- added R88: 47, Resistors_SMD:R_0805, F.Cu at (-312.4, 113.9)
- added R89: 9, Resistors_SMD:R_0805, F.Cu at (-316.5, 116.8)
- added R9: 220, Resistors_SMD:R_0805, F.Cu at (-15.7, 80.8)
- added R90: 9, Resistors_SMD:R_0805, F.Cu at (-316.5, 113.9)
- added R91: 220, Resistors_SMD:R_0805, F.Cu at (-274.2, 139.6)
- added R92: 220, Resistors_SMD:R_0805, F.Cu at (-274.2, 136.8)
- added R93: 47, Resistors_SMD:R_0805, F.Cu at (-278.3, 139.6)
- added R94: 47, Resistors_SMD:R_0805, F.Cu at (-278.3, 136.8)
- added R95: 9, Resistors_SMD:R_0805, F.Cu at (-282.5, 139.6)
- added R96: 9, Resistors_SMD:R_0805, F.Cu at (-282.5, 136.8)
- added R97: 220, Resistors_SMD:R_0805, F.Cu at (-282.5, 126.1)
- added R98: 220, Resistors_SMD:R_0805, F.Cu at (-278.3, 126.1)
- added R99: 47, Resistors_SMD:R_0805, F.Cu at (-282.5, 129.0)
- added U1: SN74AVCH16T245_DGV_48, FMC_MIPI_v2_sym:DGV48, F.Cu at (-2.10, 73.0)
- added U2: SN74AVCH16T245_DGV_48, FMC_MIPI_v2_sym:DGV48, F.Cu at (-118.4, -57.3)
- added U3: SN74AVCH16T245_DGV_48, FMC_MIPI_v2_sym:DGV48, F.Cu at (-342.9, 130.5)
- added U4: DS25BR440_RTA_40, FMC_MIPI_v2_sym:DS25BR440_SQA40A, F.Cu at (-317.8, 171.5)
- IC1, IC2: value HD3SS3411TRWARQ1 -> PI3WVR626XEBEX; footprint HD3SS3411TRWARQ1 -> QFN35P250X250X50-25N
- IC3: value PI3WVR628XBEX -> PI3WVR626XEBEX; footprint BGA24C40P4X6_170X240X50 -> QFN35P250X250X50-25N
- moved IC3 271.0 mm to (-107.8, -54.1)
- moved IC2 124.6 mm to (8.10, 69.3), turned to 90 degrees
- moved IC1 39.9 mm to (149.4, 97.2), turned to 90 degrees
Connections:
- IC1 pad 1: (no net) -> /LVDS_to_Jetson_lines/Level_shift_and_switch/sheet61A8362C/LP_CLK_N
- IC1 pad 10: (no net) -> CSI_B_D0_N
- IC1 pad 11: (no net) -> CSI_B_D1_P
- IC1 pad 12: (no net) -> CSI_B_D1_N
- IC1 pad 14: (no net) -> /LVDS_to_Jetson_lines/Level_shift_and_switch/sheet61A8362C/LP_D1_N
- IC1 pad 15: (no net) -> /LVDS_to_Jetson_lines/Level_shift_and_switch/sheet61A8362C/sheet61958BD1/SLVS_OUT_N
- IC1 pad 2: (no net) -> /LVDS_to_Jetson_lines/Level_shift_and_switch/sheet61A8362C/LVDS_2_SLVS/SLVS_OUT_N
- IC1 pad 3: (no net) -> /LVDS_to_Jetson_lines/Level_shift_and_switch/sheet61A8362C/LP_CLK_P
- IC1 pad 4: (no net) -> /LVDS_to_Jetson_lines/Level_shift_and_switch/sheet61A8362C/LVDS_2_SLVS/SLVS_OUT_P
- IC1 pad 5: (no net) -> Net-(IC1-Pad5)
- IC1 pad 6: (no net) -> CSI_B_CLK_P
- IC1 pad 7: (no net) -> CSI_B_CLK_N
- IC1 pad 8: (no net) -> CSI_B_D0_P
- IC1 pad 9: (no net) -> Earth
- IC2 pad 1: (no net) -> /LVDS_to_Jetson_lines/Level_shift_and_switch/sheet61A8362B/LP_CLK_N
- IC2 pad 10: (no net) -> CSI_A_D0_N
- IC2 pad 11: (no net) -> CSI_A_D1_P
- IC2 pad 12: (no net) -> CSI_A_D1_N
- IC2 pad 14: (no net) -> /LVDS_to_Jetson_lines/Level_shift_and_switch/sheet61A8362B/LP_D1_N
- IC2 pad 15: (no net) -> /LVDS_to_Jetson_lines/Level_shift_and_switch/sheet61A8362B/sheet61958BD1/SLVS_OUT_N
- IC2 pad 2: (no net) -> /LVDS_to_Jetson_lines/Level_shift_and_switch/sheet61A8362B/LVDS_2_SLVS/SLVS_OUT_N
- IC2 pad 3: (no net) -> /LVDS_to_Jetson_lines/Level_shift_and_switch/sheet61A8362B/LP_CLK_P
- IC2 pad 4: (no net) -> /LVDS_to_Jetson_lines/Level_shift_and_switch/sheet61A8362B/LVDS_2_SLVS/SLVS_OUT_P
- IC2 pad 5: (no net) -> Net-(IC2-Pad5)
- IC2 pad 6: (no net) -> CSI_A_CLK_P
- IC2 pad 7: (no net) -> CSI_A_CLK_N
- IC2 pad 8: (no net) -> CSI_A_D0_P
- IC2 pad 9: (no net) -> Earth
- J2 pad 1: (no net) -> CSI_A_D0_P
- J2 pad 10: (no net) -> CSI_B_CLK_N
- J2 pad 13: (no net) -> CSI_A_D1_P
- J2 pad 14: (no net) -> CSI_B_D1_P
- J2 pad 15: (no net) -> CSI_A_D1_N
- J2 pad 16: (no net) -> CSI_B_D1_N
- J2 pad 19: (no net) -> CSI_C_D0_P
- J2 pad 2: (no net) -> CSI_B_D0_P
- J2 pad 20: (no net) -> CSI_D_D0_P
- J2 pad 21: (no net) -> CSI_C_D0_N
- J2 pad 22: (no net) -> CSI_D_D0_N
- J2 pad 25: (no net) -> CSI_C_CLK_P
- J2 pad 26: (no net) -> CSI_D_CLK_P
- J2 pad 27: (no net) -> CSI_C_CLK_N
- J2 pad 28: (no net) -> CSI_D_CLK_N
- J2 pad 3: (no net) -> CSI_A_D0_N
- J2 pad 31: (no net) -> CSI_C_D1_P
- J2 pad 32: (no net) -> CSI_D_D1_P
- J2 pad 33: (no net) -> CSI_C_D1_N
- J2 pad 34: (no net) -> CSI_D_D1_N
- J2 pad 37: (no net) -> CSI_E_D0_P
- J2 pad 38: (no net) -> CSI_F_D0_P
- J2 pad 39: (no net) -> CSI_E_D0_N
- J2 pad 4: (no net) -> CSI_B_D0_N
- J2 pad 40: (no net) -> CSI_F_D0_N
- J2 pad 43: (no net) -> CSI_E_CLK_P
- J2 pad 44: (no net) -> CSI_F_CLK_P
- J2 pad 45: (no net) -> CSI_E_CLK_N
- J2 pad 46: (no net) -> CSI_F_CLK_N
- J2 pad 49: (no net) -> CSI_E_D1_P
- J2 pad 50: (no net) -> CSI_F_D1_P
- J2 pad 51: (no net) -> CSI_E_D1_N
- J2 pad 52: (no net) -> CSI_F_D1_N
- J2 pad 7: (no net) -> CSI_A_CLK_P
- J2 pad 8: (no net) -> CSI_B_CLK_P
- J2 pad 9: (no net) -> CSI_A_CLK_N
Other:
- net class Default: clearance 0.2 -> 0.1016; trace_width 0.25 -> 0.1016
- rule trace_clearance: 0.2 -> 0.1016
- rule trace_min: 0.2 -> 0.1016

Commit message: good, added re-driver
Parts:
- removed C17, C18, C19, C20, C21, C23, C27, C28, C29, C30: 0.1uF, Capacitors_SMD:C_0402
- removed C22, C24: 0.01uF, Capacitors_SMD:C_0402
- removed C25, C26: 1uF, Capacitors_SMD:C_0603
- removed IC1, IC2, IC3, IC4, IC5, IC6: PI3WVR626XEBEX, QFN35P250X250X50-25N
- removed R100, R106, R107, R112, R113, R118, R119, R23, R24, R29, R30, R35, R36, R42, R43, R48, R49, R54, R55, R61, R62, R67, R68, R73, R74, R79, R80, R87, R88, R93, R94, R99: 47, Resistors_SMD:R_0805
- removed R101, R102, R108, R109, R114, R115, R120, R121, R25, R26, R31, R32, R37, R38, R44, R45, R50, R51, R56, R57, R63, R64, R69, R70, R75, R76, R81, R82, R89, R90, R95, R96: 9, Resistors_SMD:R_0805
- removed R103, R39, R58, R84: 4.7K, Resistors_SMD:R_0805
- removed R104, R105, R110, R111, R116, R117, R21, R22, R27, R28, R33, R34, R40, R41, R46, R47, R52, R53, R59, R60, R65, R66, R71, R72, R77, R78, R85, R86, R91, R92, R97, R98: 220, Resistors_SMD:R_0805
- removed R122, R123, R126, R127, R128: 4.7k, Resistors_SMD:R_0805
- removed R124, R125: 2.2k, Resistors_SMD:R_0805
- removed R83: 100, Resistors_SMD:R_0805
- C1, C2, C3, C4: moved to F.Cu
- C11, C12, C5: value 0.1uF -> 1uF; footprint Capacitors_SMD:C_0402 -> Capacitors_SMD:C_0603
- C14, C16, C8: value 0.01uF -> 0.1uF
- C6: value 0.01uF -> 1uF; footprint Capacitors_SMD:C_0402 -> Capacitors_SMD:C_0603
- R1: value 4.7K -> 0; moved to B.Cu
- R10, R11, R16, R4: value 47 -> 4.7k
- R12, R13, R18, R19, R6: value 9 -> 2.2k
- R14, R15, R3, R8, R9: value 220 -> 4.7k
- R17, R5: value 47 -> 2.2k
- R2: value 220 -> 0; moved to B.Cu
- R20: value 4.7K -> 2.2k
- R7: value 9 -> 4.7k
- U1: moved to B.Cu
- U2: value SN74AVCH16T245_DGV_48 -> TS3DDR3812_RUA_42; footprint FMC_MIPI_v2_sym:DGV48 -> FMC_MIPI_v2_sym:TS3DDR3812RUAR
- U3: value SN74AVCH16T245_DGV_48 -> DS25BR440_RTA_40; footprint FMC_MIPI_v2_sym:DGV48 -> FMC_MIPI_v2_sym:DS25BR440_SQA40A
- moved U3 263.8 mm to (-105.5, 15.6)
- moved U4 248.9 mm to (-104.8, 42.6)
- moved C5 137.9 mm to (-112.4, 15.7)
- moved C6 133.6 mm to (-99.4, 16.0), turned to 180 degrees
- moved C8 132.7 mm to (-112.3, 12.9)
- moved R5 126.8 mm to (-111.8, 7.60), turned to 270 degrees
- moved R8 119.9 mm to (-108.5, 7.65), turned to 90 degrees
- moved C7 118.0 mm to (-105.8, 22.4), turned to 90 degrees
- moved R17 116.9 mm to (-111.2, 23.0), turned to 90 degrees
- moved R6 115.7 mm to (-99.5, 7.70), turned to 270 degrees
- moved R7 113.8 mm to (-105.1, 7.70), turned to 90 degrees
- moved R9 113.7 mm to (-102.8, 7.65), turned to 270 degrees
- moved R18 110.3 mm to (-100.0, 23.0), turned to 90 degrees
- moved R3 109.3 mm to (-108.1, 22.9), turned to 270 degrees
- moved R20 108.5 mm to (-100.6, 49.6), turned to 90 degrees
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Connections:
- C1 pad 1: /LVDS_to_Jetson_lines/SWITCH_VDD_VADJ -> /LVDS_to_Jetson_lines/VDD_VADJ
- C10 pad 1: /LVDS_to_Jetson_lines/SWITCH_VDD_VADJ -> Earth
- C10 pad 2: Earth -> /LVDS_to_Jetson_lines/VOLT_3P3
- C11 pad 1: /LVDS_to_Jetson_lines/VOLT_1P2 -> Earth
- C11 pad 2: Earth -> /LVDS_to_Jetson_lines/VOLT_3P3
- C12 pad 1: /LVDS_to_Jetson_lines/VOLT_1P2 -> Earth
- C12 pad 2: Earth -> /LVDS_to_Jetson_lines/VOLT_3P3
- C13 pad 2: /LVDS_to_Jetson_lines/SWITCH_VDD_VADJ -> /LVDS_to_Jetson_lines/VOLT_3P3
- C14 pad 2: /LVDS_to_Jetson_lines/SWITCH_VDD_VADJ -> /LVDS_to_Jetson_lines/VOLT_3P3
- C15 pad 2: /LVDS_to_Jetson_lines/SWITCH_VDD_VADJ -> /LVDS_to_Jetson_lines/VOLT_3P3
- C16 pad 2: /LVDS_to_Jetson_lines/SWITCH_VDD_VADJ -> /LVDS_to_Jetson_lines/VOLT_3P3
- C2 pad 1: /LVDS_to_Jetson_lines/SWITCH_VDD_VADJ -> /LVDS_to_Jetson_lines/VDD_VADJ
- C5 pad 2: /LVDS_to_Jetson_lines/SWITCH_VDD_VADJ -> /LVDS_to_Jetson_lines/VOLT_3P3
- C6 pad 2: /LVDS_to_Jetson_lines/SWITCH_VDD_VADJ -> /LVDS_to_Jetson_lines/VOLT_3P3
- C7 pad 2: /LVDS_to_Jetson_lines/SWITCH_VDD_VADJ -> /LVDS_to_Jetson_lines/VOLT_3P3
- C8 pad 2: /LVDS_to_Jetson_lines/SWITCH_VDD_VADJ -> /LVDS_to_Jetson_lines/VOLT_3P3
- C9 pad 1: /LVDS_to_Jetson_lines/SWITCH_VDD_VADJ -> Earth
- C9 pad 2: Earth -> /LVDS_to_Jetson_lines/VOLT_3P3
- J2 pad 19: CSI_C_D0_P -> (no net)
- J2 pad 20: CSI_D_D0_P -> (no net)
- J2 pad 21: CSI_C_D0_N -> (no net)
- J2 pad 22: CSI_D_D0_N -> (no net)
- J2 pad 25: CSI_C_CLK_P -> (no net)
- J2 pad 26: CSI_D_CLK_P -> (no net)
- J2 pad 27: CSI_C_CLK_N -> (no net)
- J2 pad 28: CSI_D_CLK_N -> (no net)
- J2 pad 31: CSI_C_D1_P -> (no net)
- J2 pad 32: CSI_D_D1_P -> (no net)
- J2 pad 33: CSI_C_D1_N -> (no net)
- J2 pad 34: CSI_D_D1_N -> (no net)
- J2 pad 37: CSI_E_D0_P -> (no net)
- J2 pad 38: CSI_F_D0_P -> (no net)
- J2 pad 39: CSI_E_D0_N -> (no net)
- J2 pad 40: CSI_F_D0_N -> (no net)
- J2 pad 43: CSI_E_CLK_P -> (no net)
- J2 pad 44: CSI_F_CLK_P -> (no net)
- J2 pad 45: CSI_E_CLK_N -> (no net)
- J2 pad 46: CSI_F_CLK_N -> (no net)
- J2 pad 49: CSI_E_D1_P -> (no net)
- J2 pad 50: CSI_F_D1_P -> (no net)
- J2 pad 51: CSI_E_D1_N -> (no net)
- J2 pad 52: CSI_F_D1_N -> (no net)
- R1 pad 1: Earth -> Net-(R1-Pad1)
- R1 pad 2: Net-(IC1-Pad5) -> (no net)
- R10 pad 1: /LVDS_to_Jetson_lines/Level_shift_and_switch/sheet61A8362C/sheet61958BD1/SLVS_OUT_P -> Net-(R10-Pad1)
- R10 pad 2: /LVDS_to_Jetson_lines/Level_shift_and_switch/BOT_HS_D1_P -> /LVDS_to_Jetson_lines/VOLT_3P3
- R11 pad 1: /LVDS_to_Jetson_lines/Level_shift_and_switch/sheet61A8362C/sheet61958BD1/SLVS_OUT_N -> Net-(R11-Pad1)
- R11 pad 2: /LVDS_to_Jetson_lines/Level_shift_and_switch/BOT_HS_D1_N -> /LVDS_to_Jetson_lines/VOLT_3P3
- R12 pad 1: /LVDS_to_Jetson_lines/Level_shift_and_switch/sheet61A8362C/sheet61958BD1/SLVS_OUT_P -> Earth
- R12 pad 2: Earth -> /LVDS_to_Jetson_lines/Level_shift_and_switch/sheet61B8C8AB/DS25_EQ0
- R13 pad 1: /LVDS_to_Jetson_lines/Level_shift_and_switch/sheet61A8362C/sheet61958BD1/SLVS_OUT_N -> Earth
- R13 pad 2: Earth -> /LVDS_to_Jetson_lines/Level_shift_and_switch/sheet61B8C8AB/DS25_PE0
- R14 pad 1: /LVDS_to_Jetson_lines/Level_shift_and_switch/BOT_HS_CLK_P -> /LVDS_to_Jetson_lines/VOLT_3P3
- R14 pad 2: /LVDS_to_Jetson_lines/VOLT_2P5 -> Net-(R14-Pad2)
- R15 pad 1: /LVDS_to_Jetson_lines/Level_shift_and_switch/BOT_HS_CLK_N -> /LVDS_to_Jetson_lines/VOLT_3P3
- R15 pad 2: /LVDS_to_Jetson_lines/VOLT_2P5 -> Net-(R15-Pad2)
- R16 pad 1: /LVDS_to_Jetson_lines/Level_shift_and_switch/sheet61A8362C/LVDS_2_SLVS/SLVS_OUT_P -> /LVDS_to_Jetson_lines/VOLT_3P3
- R16 pad 2: /LVDS_to_Jetson_lines/Level_shift_and_switch/BOT_HS_CLK_P -> Net-(R16-Pad2)
- R17 pad 1: /LVDS_to_Jetson_lines/Level_shift_and_switch/sheet61A8362C/LVDS_2_SLVS/SLVS_OUT_N -> Earth
- R17 pad 2: /LVDS_to_Jetson_lines/Level_shift_and_switch/BOT_HS_CLK_N -> /LVDS_to_Jetson_lines/Level_shift_and_switch/sheet61B2E685/DS25_EQ2
- R18 pad 1: /LVDS_to_Jetson_lines/Level_shift_and_switch/sheet61A8362C/LVDS_2_SLVS/SLVS_OUT_P -> Earth
- R18 pad 2: Earth -> /LVDS_to_Jetson_lines/Level_shift_and_switch/sheet61B2E685/DS25_PE1
- R19 pad 1: /LVDS_to_Jetson_lines/Level_shift_and_switch/sheet61A8362C/LVDS_2_SLVS/SLVS_OUT_N -> Earth
- R19 pad 2: Earth -> /LVDS_to_Jetson_lines/Level_shift_and_switch/sheet61B8C8AB/DS25_EQ2
- R2 pad 1: /LVDS_to_Jetson_lines/Level_shift_and_switch/BOT_HS_D0_P -> Net-(R2-Pad1)
- R2 pad 2: /LVDS_to_Jetson_lines/VOLT_2P5 -> /LVDS_to_Jetson_lines/VOLT_3P3
- R20 pad 2: Net-(IC2-Pad5) -> /LVDS_to_Jetson_lines/Level_shift_and_switch/sheet61B8C8AB/DS25_PE1
- R3 pad 1: /LVDS_to_Jetson_lines/Level_shift_and_switch/BOT_HS_D0_N -> Net-(R3-Pad1)
- R3 pad 2: /LVDS_to_Jetson_lines/VOLT_2P5 -> /LVDS_to_Jetson_lines/VOLT_3P3
- R4 pad 1: /LVDS_to_Jetson_lines/Level_shift_and_switch/sheet61A8362C/sheet61958A5A/SLVS_OUT_P -> Net-(R4-Pad1)
- R4 pad 2: /LVDS_to_Jetson_lines/Level_shift_and_switch/BOT_HS_D0_P -> /LVDS_to_Jetson_lines/VOLT_3P3
- R5 pad 1: /LVDS_to_Jetson_lines/Level_shift_and_switch/sheet61A8362C/sheet61958A5A/SLVS_OUT_N -> Earth
- R5 pad 2: /LVDS_to_Jetson_lines/Level_shift_and_switch/BOT_HS_D0_N -> /LVDS_to_Jetson_lines/Level_shift_and_switch/sheet61B2E685/DS25_EQ0
- R6 pad 1: /LVDS_to_Jetson_lines/Level_shift_and_switch/sheet61A8362C/sheet61958A5A/SLVS_OUT_P -> Earth
- R6 pad 2: Earth -> /LVDS_to_Jetson_lines/Level_shift_and_switch/sheet61B2E685/DS25_PE0
- R7 pad 1: /LVDS_to_Jetson_lines/Level_shift_and_switch/sheet61A8362C/sheet61958A5A/SLVS_OUT_N -> /LVDS_to_Jetson_lines/VOLT_3P3
- R7 pad 2: Earth -> Net-(R7-Pad2)
- R8 pad 1: /LVDS_to_Jetson_lines/Level_shift_and_switch/BOT_HS_D1_P -> /LVDS_to_Jetson_lines/VOLT_3P3
- R8 pad 2: /LVDS_to_Jetson_lines/VOLT_2P5 -> Net-(R8-Pad2)
- R9 pad 1: /LVDS_to_Jetson_lines/Level_shift_and_switch/BOT_HS_D1_N -> /LVDS_to_Jetson_lines/VOLT_3P3
- R9 pad 2: /LVDS_to_Jetson_lines/VOLT_2P5 -> Net-(R9-Pad2)
- U1 pad 18: /LVDS_to_Jetson_lines/SWITCH_VDD_VADJ -> /LVDS_to_Jetson_lines/VDD_VADJ
- U1 pad 26: /LVDS_to_Jetson_lines/Level_shift_and_switch/sheet61A8362C/LP_CLK_P -> /LVDS_to_Jetson_lines/Level_shift_and_switch/TOP_1P2_LP_D1_P
- U1 pad 27: /LVDS_to_Jetson_lines/Level_shift_and_switch/sheet61A8362C/LP_CLK_N -> /LVDS_to_Jetson_lines/Level_shift_and_switch/TOP_1P2_LP_D1_N
- U1 pad 29: /LVDS_to_Jetson_lines/Level_shift_and_switch/sheet61A8362C/LP_D0_P -> /LVDS_to_Jetson_lines/Level_shift_and_switch/TOP_1P2_LP_D0_P
- U1 pad 30: /LVDS_to_Jetson_lines/Level_shift_and_switch/sheet61A8362C/LP_D0_N -> /LVDS_to_Jetson_lines/Level_shift_and_switch/TOP_1P2_LP_D0_N
- U1 pad 32: /LVDS_to_Jetson_lines/Level_shift_and_switch/sheet61A8362C/LP_D1_P -> /LVDS_to_Jetson_lines/Level_shift_and_switch/TOP_1P2_LP_CLK_P
- U1 pad 33: /LVDS_to_Jetson_lines/Level_shift_and_switch/sheet61A8362C/LP_D1_N -> /LVDS_to_Jetson_lines/Level_shift_and_switch/TOP_1P2_LP_CLK_N
- U1 pad 40: /LVDS_to_Jetson_lines/Level_shift_and_switch/sheet61A8362B/LP_CLK_P -> /LVDS_to_Jetson_lines/Level_shift_and_switch/BOT_1P2_LP_CLK_P
- U1 pad 41: /LVDS_to_Jetson_lines/Level_shift_and_switch/sheet61A8362B/LP_CLK_N -> /LVDS_to_Jetson_lines/Level_shift_and_switch/BOT_1P2_LP_CLK_N
- U1 pad 43: /LVDS_to_Jetson_lines/Level_shift_and_switch/sheet61A8362B/LP_D0_P -> /LVDS_to_Jetson_lines/Level_shift_and_switch/BOT_1P2_LP_D0_P
- U1 pad 44: /LVDS_to_Jetson_lines/Level_shift_and_switch/sheet61A8362B/LP_D0_N -> /LVDS_to_Jetson_lines/Level_shift_and_switch/BOT_1P2_LP_D0_N
- U1 pad 46: /LVDS_to_Jetson_lines/Level_shift_and_switch/sheet61A8362B/LP_D1_P -> /LVDS_to_Jetson_lines/Level_shift_and_switch/BOT_1P2_LP_D1_P
- U1 pad 47: /LVDS_to_Jetson_lines/Level_shift_and_switch/sheet61A8362B/LP_D1_N -> /LVDS_to_Jetson_lines/Level_shift_and_switch/BOT_1P2_LP_D1_N
- U1 pad 7: /LVDS_to_Jetson_lines/SWITCH_VDD_VADJ -> /LVDS_to_Jetson_lines/VDD_VADJ
- U2 pad 1: Earth -> /LVDS_to_Jetson_lines/VOLT_3P3
- U2 pad 10: Earth -> Net-(R1-Pad1)
- U2 pad 11: Earth -> CSI_A_CLK_N
- U2 pad 12: Earth -> CSI_A_CLK_P
- U2 pad 13: Earth -> CSI_A_D0_N
- U2 pad 14: Earth -> CSI_A_D0_P
- U2 pad 15: Earth -> CSI_A_D1_N
- U2 pad 16: (no net) -> CSI_A_D1_P
- U2 pad 17: (no net) -> /LVDS_to_Jetson_lines/VOLT_3P3
- U2 pad 18: /LVDS_to_Jetson_lines/SWITCH_VDD_VADJ -> /LVDS_to_Jetson_lines/Level_shift_and_switch/TOP_1P2_LP_D1_P
- U2 pad 19: (no net) -> /LVDS_to_Jetson_lines/Level_shift_and_switch/TOP_RDR_HS_D1_P
- U2 pad 2: (no net) -> CSI_B_D1_N
- U2 pad 20: (no net) -> /LVDS_to_Jetson_lines/Level_shift_and_switch/TOP_1P2_LP_D1_N
- U2 pad 21: Earth -> /LVDS_to_Jetson_lines/Level_shift_and_switch/TOP_RDR_HS_D1_N
- U2 pad 22: (no net) -> /LVDS_to_Jetson_lines/Level_shift_and_switch/TOP_1P2_LP_D0_P
- U2 pad 23: (no net) -> /LVDS_to_Jetson_lines/Level_shift_and_switch/TOP_RDR_HS_D0_P
- U2 pad 24: Earth -> /LVDS_to_Jetson_lines/Level_shift_and_switch/TOP_1P2_LP_D0_N
- U2 pad 25: Earth -> /LVDS_to_Jetson_lines/Level_shift_and_switch/TOP_RDR_HS_D0_N
- U2 pad 26: /LVDS_to_Jetson_lines/sheet61A38142/sheet61A8362C/LP_CLK_P -> /LVDS_to_Jetson_lines/Level_shift_and_switch/TOP_1P2_LP_CLK_P
- U2 pad 27: /LVDS_to_Jetson_lines/sheet61A38142/sheet61A8362C/LP_CLK_N -> /LVDS_to_Jetson_lines/Level_shift_and_switch/TOP_RDR_HS_CLK_P
- U2 pad 28: Earth -> /LVDS_to_Jetson_lines/Level_shift_and_switch/TOP_1P2_LP_CLK_N
- U2 pad 29: /LVDS_to_Jetson_lines/sheet61A38142/sheet61A8362C/LP_D0_P -> /LVDS_to_Jetson_lines/Level_shift_and_switch/TOP_RDR_HS_CLK_N
- U2 pad 3: (no net) -> CSI_B_D1_P
- U2 pad 30: /LVDS_to_Jetson_lines/sheet61A38142/sheet61A8362C/LP_D0_N -> /LVDS_to_Jetson_lines/VOLT_3P3
- U2 pad 31: /LVDS_to_Jetson_lines/VOLT_1P2 -> /LVDS_to_Jetson_lines/Level_shift_and_switch/BOT_1P2_LP_CLK_P
- U2 pad 32: /LVDS_to_Jetson_lines/sheet61A38142/sheet61A8362C/LP_D1_P -> /LVDS_to_Jetson_lines/Level_shift_and_switch/BOT_RDR_HS_CLK_P
- U2 pad 33: /LVDS_to_Jetson_lines/sheet61A38142/sheet61A8362C/LP_D1_N -> /LVDS_to_Jetson_lines/Level_shift_and_switch/BOT_1P2_LP_CLK_N
- U2 pad 34: Earth -> /LVDS_to_Jetson_lines/Level_shift_and_switch/BOT_RDR_HS_CLK_N
- U2 pad 35: Earth -> /LVDS_to_Jetson_lines/Level_shift_and_switch/BOT_1P2_LP_D0_P
- U2 pad 36: Earth -> /LVDS_to_Jetson_lines/Level_shift_and_switch/BOT_RDR_HS_D0_P
- U2 pad 37: Earth -> /LVDS_to_Jetson_lines/Level_shift_and_switch/BOT_1P2_LP_D0_N
- U2 pad 38: Earth -> /LVDS_to_Jetson_lines/Level_shift_and_switch/BOT_RDR_HS_D0_N
- U2 pad 39: Earth -> /LVDS_to_Jetson_lines/Level_shift_and_switch/BOT_RDR_HS_D1_P
- U2 pad 4: Earth -> CSI_B_D0_N
- U2 pad 40: /LVDS_to_Jetson_lines/sheet61A38142/sheet61A8362B/LP_CLK_P -> /LVDS_to_Jetson_lines/Level_shift_and_switch/BOT_1P2_LP_D1_P
- U2 pad 41: /LVDS_to_Jetson_lines/sheet61A38142/sheet61A8362B/LP_CLK_N -> /LVDS_to_Jetson_lines/Level_shift_and_switch/BOT_RDR_HS_D1_N
- U2 pad 42: /LVDS_to_Jetson_lines/VOLT_1P2 -> /LVDS_to_Jetson_lines/Level_shift_and_switch/BOT_1P2_LP_D1_N
- U2 pad 43: /LVDS_to_Jetson_lines/sheet61A38142/sheet61A8362B/LP_D0_P -> Earth
- U2 pad 5: (no net) -> CSI_B_D0_P
- U2 pad 6: (no net) -> CSI_B_CLK_N
- U2 pad 7: /LVDS_to_Jetson_lines/SWITCH_VDD_VADJ -> CSI_B_CLK_P
- U2 pad 8: (no net) -> Net-(R2-Pad1)
- U2 pad 9: (no net) -> Net-(R1-Pad1)
- U3 pad 1: Earth -> (no net)
- U3 pad 10: Earth -> (no net)
- U3 pad 11: Earth -> /LVDS_to_Jetson_lines/Level_shift_and_switch/sheet61B2E685/DS25_EQ2
- U3 pad 12: Earth -> /LVDS_to_Jetson_lines/Level_shift_and_switch/sheet61B2E685/DS25_EQ2
- U3 pad 13: Earth -> Net-(R3-Pad1)
- U3 pad 14: Earth -> Net-(R4-Pad1)
- U3 pad 15: Earth -> /LVDS_to_Jetson_lines/VOLT_3P3
- U3 pad 16: (no net) -> Earth
- U3 pad 18: /LVDS_to_Jetson_lines/SWITCH_VDD_VADJ -> /LVDS_to_Jetson_lines/Level_shift_and_switch/sheet61B2E685/DS25_PE1
- U3 pad 19: (no net) -> /LVDS_to_Jetson_lines/Level_shift_and_switch/sheet61B2E685/DS25_PE1
- U3 pad 20: (no net) -> /LVDS_to_Jetson_lines/Level_shift_and_switch/sheet61B2E685/DS25_PE1
- U3 pad 21: Earth -> /LVDS_to_Jetson_lines/Level_shift_and_switch/TOP_RDR_HS_CLK_N
- U3 pad 22: (no net) -> /LVDS_to_Jetson_lines/Level_shift_and_switch/TOP_RDR_HS_CLK_P
- U3 pad 23: (no net) -> /LVDS_to_Jetson_lines/Level_shift_and_switch/TOP_RDR_HS_D0_N
- U3 pad 24: Earth -> /LVDS_to_Jetson_lines/Level_shift_and_switch/TOP_RDR_HS_D0_P
- U3 pad 25: Earth -> /LVDS_to_Jetson_lines/VOLT_3P3
- U3 pad 26: /LVDS_to_Jetson_lines/Redriver_L_shift_and_switch/sheet61A8362C/LP_D1_N -> /LVDS_to_Jetson_lines/Level_shift_and_switch/TOP_RDR_HS_D1_N
- U3 pad 27: /LVDS_to_Jetson_lines/Redriver_L_shift_and_switch/sheet61A8362C/LP_D1_P -> /LVDS_to_Jetson_lines/Level_shift_and_switch/TOP_RDR_HS_D1_P
- U3 pad 28: Earth -> (no net)
- U3 pad 29: /LVDS_to_Jetson_lines/Redriver_L_shift_and_switch/sheet61A8362C/LP_D0_N -> (no net)
- U3 pad 3: (no net) -> /LVDS_to_Jetson_lines/VOLT_3P3
- U3 pad 30: /LVDS_to_Jetson_lines/Redriver_L_shift_and_switch/sheet61A8362C/LP_D0_P -> /LVDS_to_Jetson_lines/VOLT_3P3
- U3 pad 31: /LVDS_to_Jetson_lines/VOLT_1P2 -> /LVDS_to_Jetson_lines/Level_shift_and_switch/sheet61B2E685/DS25_PE0
- U3 pad 32: /LVDS_to_Jetson_lines/Redriver_L_shift_and_switch/sheet61A8362C/LP_CLK_N -> Net-(R8-Pad2)
- U3 pad 33: /LVDS_to_Jetson_lines/Redriver_L_shift_and_switch/sheet61A8362C/LP_CLK_P -> Net-(R8-Pad2)
- U3 pad 34: Earth -> Net-(R8-Pad2)
- U3 pad 35: Earth -> Net-(R8-Pad2)
- U3 pad 36: Earth -> Net-(R9-Pad2)
- U3 pad 37: Earth -> Net-(R7-Pad2)
- U3 pad 38: Earth -> Net-(R8-Pad2)
- U3 pad 39: Earth -> /LVDS_to_Jetson_lines/Level_shift_and_switch/sheet61B2E685/DS25_EQ0
- U3 pad 4: Earth -> (no net)
- U3 pad 40: /LVDS_to_Jetson_lines/Redriver_L_shift_and_switch/sheet61A8362B/LP_D1_N -> /LVDS_to_Jetson_lines/Level_shift_and_switch/sheet61B2E685/DS25_EQ0
- U3 pad 41: /LVDS_to_Jetson_lines/Redriver_L_shift_and_switch/sheet61A8362B/LP_D1_P -> Earth
- U3 pad 7: /LVDS_to_Jetson_lines/SWITCH_VDD_VADJ -> (no net)
- U3 pad 8: (no net) -> /LVDS_to_Jetson_lines/VOLT_3P3
- U4 pad 11: /LVDS_to_Jetson_lines/Redriver_L_shift_and_switch/sheet61BA18CE/DS25_EQ0 -> /LVDS_to_Jetson_lines/Level_shift_and_switch/sheet61B8C8AB/DS25_EQ2
- U4 pad 12: /LVDS_to_Jetson_lines/Redriver_L_shift_and_switch/sheet61BA18CE/DS25_EQ0 -> /LVDS_to_Jetson_lines/Level_shift_and_switch/sheet61B8C8AB/DS25_EQ2
- U4 pad 13: Net-(R122-Pad1) -> Net-(R10-Pad1)
- U4 pad 14: Net-(R123-Pad1) -> Net-(R11-Pad1)
- U4 pad 18: /LVDS_to_Jetson_lines/Redriver_L_shift_and_switch/sheet61BA18CE/DS25_PE0 -> /LVDS_to_Jetson_lines/Level_shift_and_switch/sheet61B8C8AB/DS25_PE1
- U4 pad 19: /LVDS_to_Jetson_lines/Redriver_L_shift_and_switch/sheet61BA18CE/DS25_PE0 -> /LVDS_to_Jetson_lines/Level_shift_and_switch/sheet61B8C8AB/DS25_PE1
- U4 pad 20: /LVDS_to_Jetson_lines/Redriver_L_shift_and_switch/sheet61BA18CE/DS25_PE0 -> /LVDS_to_Jetson_lines/Level_shift_and_switch/sheet61B8C8AB/DS25_PE1
- U4 pad 21: /LVDS_to_Jetson_lines/Redriver_L_shift_and_switch/sheet61A8362B/HS_D1_N -> /LVDS_to_Jetson_lines/Level_shift_and_switch/BOT_RDR_HS_D1_N
- U4 pad 22: /LVDS_to_Jetson_lines/Redriver_L_shift_and_switch/sheet61A8362B/HS_D1_P -> /LVDS_to_Jetson_lines/Level_shift_and_switch/BOT_RDR_HS_D1_P
- U4 pad 23: /LVDS_to_Jetson_lines/Redriver_L_shift_and_switch/sheet61A8362B/HS_D0_N -> /LVDS_to_Jetson_lines/Level_shift_and_switch/BOT_RDR_HS_D0_N
- U4 pad 24: /LVDS_to_Jetson_lines/Redriver_L_shift_and_switch/sheet61A8362B/HS_D0_P -> /LVDS_to_Jetson_lines/Level_shift_and_switch/BOT_RDR_HS_D0_P
- U4 pad 26: /LVDS_to_Jetson_lines/Redriver_L_shift_and_switch/sheet61A8362B/HS_CLK_N -> /LVDS_to_Jetson_lines/Level_shift_and_switch/BOT_RDR_HS_CLK_N
- U4 pad 27: /LVDS_to_Jetson_lines/Redriver_L_shift_and_switch/sheet61A8362B/HS_CLK_P -> /LVDS_to_Jetson_lines/Level_shift_and_switch/BOT_RDR_HS_CLK_P
- U4 pad 28: /LVDS_to_Jetson_lines/Redriver_L_shift_and_switch/REDRIVER_TEST_TOP_OUT_N -> (no net)
- U4 pad 29: /LVDS_to_Jetson_lines/Redriver_L_shift_and_switch/REDRIVER_TEST_TOP_OUT_P -> (no net)
- U4 pad 31: /LVDS_to_Jetson_lines/Redriver_L_shift_and_switch/sheet61BA18CE/DS25_PE0 -> /LVDS_to_Jetson_lines/Level_shift_and_switch/sheet61B8C8AB/DS25_PE0
- U4 pad 32: Net-(R127-Pad2) -> Net-(R15-Pad2)
- U4 pad 33: Net-(R127-Pad2) -> Net-(R15-Pad2)
- U4 pad 34: Net-(R127-Pad2) -> Net-(R15-Pad2)
- U4 pad 35: Net-(R127-Pad2) -> Net-(R15-Pad2)
- U4 pad 36: Net-(R128-Pad2) -> Net-(R16-Pad2)
- U4 pad 37: Net-(R126-Pad2) -> Net-(R14-Pad2)
- U4 pad 38: Net-(R127-Pad2) -> Net-(R15-Pad2)
- U4 pad 39: /LVDS_to_Jetson_lines/Redriver_L_shift_and_switch/sheet61BA18CE/DS25_EQ0 -> /LVDS_to_Jetson_lines/Level_shift_and_switch/sheet61B8C8AB/DS25_EQ0
- U4 pad 40: /LVDS_to_Jetson_lines/Redriver_L_shift_and_switch/sheet61BA18CE/DS25_EQ0 -> /LVDS_to_Jetson_lines/Level_shift_and_switch/sheet61B8C8AB/DS25_EQ0
Other:
- net class Default: trace_width 0.1016 -> 0.1524; via_dia 0.8 -> 0.4064; via_drill 0.4 -> 0.3048

Commit message: good, before reducing
Parts:
- added C17: 0.1uF, Capacitors_SMD:C_0402, F.Cu at (-72.4, 30.4)
- added C18: 0.1uF, Capacitors_SMD:C_0402, F.Cu at (-63.2, 25.6)
- added C19: 0.1uF, Capacitors_SMD:C_0402, F.Cu at (-63.1, 36.5)
- added R27: 220, Resistors_SMD:R_0805, F.Cu at (-111.9, 5.71)
- added R28: 220, Resistors_SMD:R_0805, F.Cu at (-111.9, 8.59)
- added R29: 47, Resistors_SMD:R_0805, F.Cu at (-107.8, 5.71)
- added R30: 47, Resistors_SMD:R_0805, F.Cu at (-107.8, 8.59)
- added R31: 12, Resistors_SMD:R_0805, F.Cu at (-103.6, 5.71)
- added R32: 12, Resistors_SMD:R_0805, F.Cu at (-103.6, 8.59)
- added R33: 220, Resistors_SMD:R_0805, F.Cu at (-103.6, 17.6)
- added R34: 220, Resistors_SMD:R_0805, F.Cu at (-111.9, 14.7)
- added R35: 47, Resistors_SMD:R_0805, F.Cu at (-103.6, 14.7)
- added R36: 47, Resistors_SMD:R_0805, F.Cu at (-107.7, 17.6)
- added R37: 12, Resistors_SMD:R_0805, F.Cu at (-107.7, 14.7)
- added R38: 12, Resistors_SMD:R_0805, F.Cu at (-111.9, 17.6)
- added R39: 220, Resistors_SMD:R_0805, F.Cu at (-112.1, 24.4)
- added R40: 220, Resistors_SMD:R_0805, F.Cu at (-112.1, 27.3)
- added R41: 47, Resistors_SMD:R_0805, F.Cu at (-107.9, 24.4)
- added R42: 47, Resistors_SMD:R_0805, F.Cu at (-107.9, 27.3)
- added R43: 12, Resistors_SMD:R_0805, F.Cu at (-103.8, 24.4)
- added R44: 12, Resistors_SMD:R_0805, F.Cu at (-103.8, 27.3)
- added R51: 220, Resistors_SMD:R_0805, F.Cu at (-109.1, 35.1)
- added R52: 220, Resistors_SMD:R_0805, F.Cu at (-109.1, 38.0)
- added R53: 47, Resistors_SMD:R_0805, F.Cu at (-104.9, 35.1)
- added R54: 47, Resistors_SMD:R_0805, F.Cu at (-104.9, 38.0)
- added R55: 12, Resistors_SMD:R_0805, F.Cu at (-100.8, 35.1)
- added R56: 12, Resistors_SMD:R_0805, F.Cu at (-100.8, 38.0)
- added R57: 220, Resistors_SMD:R_0805, F.Cu at (-100.9, 44.7)
- added R58: 220, Resistors_SMD:R_0805, F.Cu at (-109.1, 47.6)
- added R59: 47, Resistors_SMD:R_0805, F.Cu at (-100.8, 47.6)
- added R60: 47, Resistors_SMD:R_0805, F.Cu at (-105.0, 44.7)
- added R61: 12, Resistors_SMD:R_0805, F.Cu at (-105.0, 47.6)
- added R62: 12, Resistors_SMD:R_0805, F.Cu at (-109.2, 44.7)
- added R63: 220, Resistors_SMD:R_0805, F.Cu at (-109.6, 52.0)
- added R64: 220, Resistors_SMD:R_0805, F.Cu at (-109.8, 56.3)
- added R65: 47, Resistors_SMD:R_0805, F.Cu at (-106.0, 52.9)
- added R66: 47, Resistors_SMD:R_0805, F.Cu at (-106.0, 55.6)
- added R67: 12, Resistors_SMD:R_0805, F.Cu at (-102.2, 51.6)
- added R68: 12, Resistors_SMD:R_0805, F.Cu at (-102.5, 56.3)
- added U5: SN74LV1T34DBV, TO_SOT_Packages_SMD:SOT-23-5, B.Cu at (-67.6, 16.4)
- moved R15 22.5 mm to (-129.8, 32.5)
- moved C13 22.5 mm to (-125.8, 47.5)
- moved C15 22.5 mm to (-133.8, 37.6)
- moved C16 22.5 mm to (-121.6, 39.1)
- moved R10 22.5 mm to (-130.8, 48.2)
- moved R12 22.5 mm to (-132.9, 32.6)
- moved R13 22.5 mm to (-120.2, 32.6)
- moved R14 22.5 mm to (-126.9, 32.5)
- moved R16 22.5 mm to (-123.5, 32.4)
- moved R20 22.5 mm to (-123.0, 48.0)
- moved U4 22.5 mm to (-127.3, 41.0)
- moved C11 22.5 mm to (-121.2, 41.0)
- moved C12 22.5 mm to (-134.2, 39.6)
- moved C14 22.5 mm to (-133.8, 41.9)
- moved R11 22.5 mm to (-127.8, 48.0)
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Connections:
- J2 pad 1: CSI_A_D0_P -> (no net)
- J2 pad 10: CSI_B_CLK_N -> (no net)
- J2 pad 13: CSI_A_D1_P -> (no net)
- J2 pad 14: CSI_B_D1_P -> (no net)
- J2 pad 15: CSI_A_D1_N -> (no net)
- J2 pad 16: CSI_B_D1_N -> (no net)
- J2 pad 19: (no net) -> CSI_C_D0_P
- J2 pad 2: CSI_B_D0_P -> (no net)
- J2 pad 20: (no net) -> CSI_D_D0_P
- J2 pad 21: (no net) -> CSI_C_D0_N
- J2 pad 22: (no net) -> CSI_D_D0_N
- J2 pad 25: (no net) -> CSI_C_CLK_P
- J2 pad 26: (no net) -> CSI_D_CLK_P
- J2 pad 27: (no net) -> CSI_C_CLK_N
- J2 pad 28: (no net) -> CSI_D_CLK_N
- J2 pad 3: CSI_A_D0_N -> (no net)
- J2 pad 31: (no net) -> CSI_C_D1_P
- J2 pad 32: (no net) -> CSI_D_D1_P
- J2 pad 33: (no net) -> CSI_C_D1_N
- J2 pad 34: (no net) -> CSI_D_D1_N
- J2 pad 4: CSI_B_D0_N -> (no net)
- J2 pad 7: CSI_A_CLK_P -> (no net)
- J2 pad 8: CSI_B_CLK_P -> (no net)
- J2 pad 9: CSI_A_CLK_N -> (no net)
- R1 pad 2: (no net) -> /LVDS_to_Jetson_lines/Level_shift_and_switch/SWITCH_HS_0_LP_1_3V3
- U2 pad 11: CSI_A_CLK_N -> CSI_C_CLK_N
- U2 pad 12: CSI_A_CLK_P -> CSI_C_CLK_P
- U2 pad 13: CSI_A_D0_N -> CSI_C_D0_N
- U2 pad 14: CSI_A_D0_P -> CSI_C_D0_P
- U2 pad 15: CSI_A_D1_N -> CSI_C_D1_N
- U2 pad 16: CSI_A_D1_P -> CSI_C_D1_P
- U2 pad 2: CSI_B_D1_N -> CSI_D_D1_N
- U2 pad 3: CSI_B_D1_P -> CSI_D_D1_P
- U2 pad 4: CSI_B_D0_N -> CSI_D_D0_N
- U2 pad 5: CSI_B_D0_P -> CSI_D_D0_P
- U2 pad 6: CSI_B_CLK_N -> CSI_D_CLK_N
- U2 pad 7: CSI_B_CLK_P -> CSI_D_CLK_P
- U3 pad 21: /LVDS_to_Jetson_lines/Level_shift_and_switch/TOP_RDR_HS_CLK_N -> /LVDS_to_Jetson_lines/Level_shift_and_switch/sheet61B2E685/sheet61CCEEAC/LVDS_IN_N
- U3 pad 22: /LVDS_to_Jetson_lines/Level_shift_and_switch/TOP_RDR_HS_CLK_P -> /LVDS_to_Jetson_lines/Level_shift_and_switch/sheet61B2E685/sheet61CCEEAC/LVDS_IN_P
- U3 pad 23: /LVDS_to_Jetson_lines/Level_shift_and_switch/TOP_RDR_HS_D0_N -> /LVDS_to_Jetson_lines/Level_shift_and_switch/sheet61B2E685/sheet61CC9F81/LVDS_IN_N
- U3 pad 24: /LVDS_to_Jetson_lines/Level_shift_and_switch/TOP_RDR_HS_D0_P -> /LVDS_to_Jetson_lines/Level_shift_and_switch/sheet61B2E685/sheet61CC9F81/LVDS_IN_P
- U3 pad 26: /LVDS_to_Jetson_lines/Level_shift_and_switch/TOP_RDR_HS_D1_N -> /LVDS_to_Jetson_lines/Level_shift_and_switch/sheet61B2E685/sheet61CC513F/LVDS_IN_N
- U3 pad 27: /LVDS_to_Jetson_lines/Level_shift_and_switch/TOP_RDR_HS_D1_P -> /LVDS_to_Jetson_lines/Level_shift_and_switch/sheet61B2E685/sheet61CC513F/LVDS_IN_P
- U4 pad 21: /LVDS_to_Jetson_lines/Level_shift_and_switch/BOT_RDR_HS_D1_N -> /LVDS_to_Jetson_lines/Level_shift_and_switch/sheet61B8C8AB/sheet61CCEEAC/LVDS_IN_N
- U4 pad 22: /LVDS_to_Jetson_lines/Level_shift_and_switch/BOT_RDR_HS_D1_P -> /LVDS_to_Jetson_lines/Level_shift_and_switch/sheet61B8C8AB/sheet61CCEEAC/LVDS_IN_P
- U4 pad 23: /LVDS_to_Jetson_lines/Level_shift_and_switch/BOT_RDR_HS_D0_N -> /LVDS_to_Jetson_lines/Level_shift_and_switch/sheet61B8C8AB/sheet61CC9F81/LVDS_IN_N
- U4 pad 24: /LVDS_to_Jetson_lines/Level_shift_and_switch/BOT_RDR_HS_D0_P -> /LVDS_to_Jetson_lines/Level_shift_and_switch/sheet61B8C8AB/sheet61CC9F81/LVDS_IN_P
- U4 pad 26: /LVDS_to_Jetson_lines/Level_shift_and_switch/BOT_RDR_HS_CLK_N -> /LVDS_to_Jetson_lines/Level_shift_and_switch/sheet61B8C8AB/sheet61CC513F/LVDS_IN_N
- U4 pad 27: /LVDS_to_Jetson_lines/Level_shift_and_switch/BOT_RDR_HS_CLK_P -> /LVDS_to_Jetson_lines/Level_shift_and_switch/sheet61B8C8AB/sheet61CC513F/LVDS_IN_P
