File: FMC_MIPI_v2.kicad_pcb (KiCad board)
At the start: 6 copper layers, 69 x 112 mm, 82 parts, among them J1 ASP-134488-01, J2 QTH-060-01-L-D-A, U1 SN74AVCH16T245_DGV_48, U2 TS3DDR3812_RUA_42, U3 DS25BR440_RTA_40, U4 DS25BR440_RTA_40, U5 SN74LV1T34DBV

Commit message: before re-arranging
Parts:
- removed C14, C15, C16, C17, C18, C19: 0.1uF, Capacitors_SMD:C_0402
- removed R62, R67, R68: 12, Resistors_SMD:R_0805
- removed R63, R64: 220, Resistors_SMD:R_0805
- removed R65, R66: 47, Resistors_SMD:R_0805
- added R21: 47, Resistors_SMD:R_0603, F.Cu at (-100.6, 17.8)
- added R22: 12, Resistors_SMD:R_0805, F.Cu at (-98.0, 14.7)
- added R23: 12, Resistors_SMD:R_0805, F.Cu at (-98.0, 18.8)
- added R24: 220, Resistors_SMD:R_0603, F.Cu at (-103.1, 23.9)
- added R25: 220, Resistors_SMD:R_0603, F.Cu at (-103.1, 26.9)
- added R26: 47, Resistors_SMD:R_0603, F.Cu at (-100.6, 24.4)
- added R45: 220, Resistors_SMD:R_0603, F.Cu at (-53.3, 83.8)
- added R46: 47, Resistors_SMD:R_0603, F.Cu at (-50.8, 81.3)
- added R47: 47, Resistors_SMD:R_0603, F.Cu at (-50.8, 83.3)
- added R48: 10, Resistors_SMD:R_1206_HandSoldering, F.Cu at (-47.8, 78.2)
- added R49: 10, Resistors_SMD:R_1206_HandSoldering, F.Cu at (-47.8, 86.4)
- added R50: 220, Resistors_SMD:R_0603, F.Cu at (-46.7, 93.0)
- C11, C12, C5, C6: value 1uF -> 0.1uF; footprint Capacitors_SMD:C_0603 -> Capacitors_SMD:C_0402
- C8, C9: value 0.1uF -> 1uF; footprint Capacitors_SMD:C_0402 -> Capacitors_SMD:C_0603
- R12, R13, R18, R19: value 2.2k -> 220; footprint Resistors_SMD:R_0805 -> Resistors_SMD:R_0603
- R14, R15: value 4.7k -> 47; footprint Resistors_SMD:R_0805 -> Resistors_SMD:R_0603
- R16: value 4.7k -> 12
- R17: value 2.2k -> 12
- R20: value 2.2k -> 47; footprint Resistors_SMD:R_0805 -> Resistors_SMD:R_0603
- R27, R33, R39, R40, R52, R58: value 220 -> 47; footprint Resistors_SMD:R_0805 -> Resistors_SMD:R_0603
- R28: value 220 -> 12
- R29: value 47 -> 12
- R3, R4: value 4.7k -> 2.2k
- R30: value 47 -> 220; footprint Resistors_SMD:R_0805 -> Resistors_SMD:R_0603
- R31, R37, R38, R44, R56: value 12 -> 220; footprint Resistors_SMD:R_0805 -> Resistors_SMD:R_0603
- R32: value 12 -> 47; footprint Resistors_SMD:R_0805 -> Resistors_SMD:R_0603
- R34: value 220 -> 10; footprint Resistors_SMD:R_0805 -> Resistors_SMD:R_1206_HandSoldering
- R35, R41, R42, R54, R60: value 47 -> 10; footprint Resistors_SMD:R_0805 -> Resistors_SMD:R_1206_HandSoldering
- R36: value 47 -> 100; footprint Resistors_SMD:R_0805 -> Resistors_SMD:R_1206_HandSoldering
- R43: value 12 -> 100; footprint Resistors_SMD:R_0805 -> Resistors_SMD:R_1206_HandSoldering
- R51, R53, R57, R59: footprint Resistors_SMD:R_0805 -> Resistors_SMD:R_0603
- R55, R61: value 12 -> 10; footprint Resistors_SMD:R_0805 -> Resistors_SMD:R_1206_HandSoldering
- U3: value DS25BR440_RTA_40 -> SN74LV1T34DBV; footprint FMC_MIPI_v2_sym:DS25BR440_SQA40A -> TO_SOT_Packages_SMD:SOT-23-5; moved to B.Cu
- U5: value SN74LV1T34DBV -> TS3DDR3812_RUA_42; footprint TO_SOT_Packages_SMD:SOT-23-5 -> FMC_MIPI_v2_sym:TS3DDR3812RUAR; moved to F.Cu
- moved U2 214.8 mm to (134.6, 103.6)
- moved R43 122.7 mm to (1.52, 87.4), turned to 270 degrees
- moved R38 117.4 mm to (-33.0, 104.6), turned to 90 degrees
- moved R37 114.6 mm to (-33.0, 101.6), turned to 90 degrees
- moved R42 113.4 mm to (-26.9, 106.7), turned to 270 degrees
- moved R39 112.7 mm to (-30.5, 102.1), turned to 180 degrees
- moved R40 112.1 mm to (-30.5, 104.1), turned to 180 degrees
- moved R41 110.5 mm to (-26.9, 99.6), turned to 270 degrees
- moved U5 96.4 mm to (-7.11, 91.4), turned to 180 degrees
- moved R61 88.3 mm to (-26.9, 88.9), turned to 270 degrees
- moved R51 87.5 mm to (-46.7, 96.5), turned to 90 degrees
- moved R55 87.4 mm to (-40.6, 98.6), turned to 270 degrees
- moved R58 87.0 mm to (-30.0, 83.8), turned to 180 degrees
- moved R60 86.2 mm to (-26.9, 81.3), turned to 270 degrees
- moved R53 86.0 mm to (-44.2, 96.0), turned to 180 degrees
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Connections:
- net /LVDS_to_Jetson_lines/Level_shift_and_switch/BOT_1P2_LP_CLK_N renamed /LVDS_to_Jetson_lines/Level_shift_and_switch_single/TOP_1P2_LP_D1_N
- C3 pad 1: /LVDS_to_Jetson_lines/VOLT_1P2 -> /LVDS_to_Jetson_lines/VOLT_3P3
- C4 pad 1: /LVDS_to_Jetson_lines/VOLT_1P2 -> /LVDS_to_Jetson_lines/VOLT_3P3
- C5 pad 1: Earth -> /LVDS_to_Jetson_lines/VOLT_3P3
- C5 pad 2: /LVDS_to_Jetson_lines/VOLT_3P3 -> Earth
- C6 pad 1: Earth -> /LVDS_to_Jetson_lines/VOLT_1P2
- C6 pad 2: /LVDS_to_Jetson_lines/VOLT_3P3 -> Earth
- C7 pad 1: Earth -> /LVDS_to_Jetson_lines/VOLT_1P2
- C7 pad 2: /LVDS_to_Jetson_lines/VOLT_3P3 -> Earth
- J2 pad 1: (no net) -> CSI_A_D0_P
- J2 pad 13: (no net) -> CSI_A_D1_P
- J2 pad 15: (no net) -> CSI_A_D1_N
- J2 pad 20: CSI_D_D0_P -> (no net)
- J2 pad 22: CSI_D_D0_N -> (no net)
- J2 pad 26: CSI_D_CLK_P -> (no net)
- J2 pad 28: CSI_D_CLK_N -> (no net)
- J2 pad 3: (no net) -> CSI_A_D0_N
- J2 pad 32: CSI_D_D1_P -> (no net)
- J2 pad 34: CSI_D_D1_N -> (no net)
- J2 pad 7: (no net) -> CSI_A_CLK_P
- J2 pad 9: (no net) -> CSI_A_CLK_N
- R1 pad 2: /LVDS_to_Jetson_lines/Level_shift_and_switch/SWITCH_HS_0_LP_1_3V3 -> /LVDS_to_Jetson_lines/Level_shift_and_switch_single/SWITCH_HS_0_LP_1_3V3
- R10 pad 1: Net-(R10-Pad1) -> /LVDS_to_Jetson_lines/VOLT_3P3
- R10 pad 2: /LVDS_to_Jetson_lines/VOLT_3P3 -> Net-(R10-Pad2)
- R11 pad 1: Net-(R11-Pad1) -> /LVDS_to_Jetson_lines/VOLT_3P3
- R11 pad 2: /LVDS_to_Jetson_lines/VOLT_3P3 -> Net-(R11-Pad2)
- R12 pad 1: Earth -> /LVDS_to_Jetson_lines/Level_shift_and_switch_single/sheet61B2E685/sheet61CC513F/LVDS_IN_P
- R12 pad 2: /LVDS_to_Jetson_lines/Level_shift_and_switch/sheet61B8C8AB/DS25_EQ0 -> /LVDS_to_Jetson_lines/VOLT_2P5
- R13 pad 1: Earth -> /LVDS_to_Jetson_lines/VOLT_2P5
- R13 pad 2: /LVDS_to_Jetson_lines/Level_shift_and_switch/sheet61B8C8AB/DS25_PE0 -> /LVDS_to_Jetson_lines/Level_shift_and_switch_single/sheet61B2E685/sheet61CC513F/LVDS_IN_N
- R14 pad 1: /LVDS_to_Jetson_lines/VOLT_3P3 -> /LVDS_to_Jetson_lines/Level_shift_and_switch_single/TOP_RDR_HS_D0_P
- R14 pad 2: Net-(R14-Pad2) -> /LVDS_to_Jetson_lines/Level_shift_and_switch_single/sheet61B2E685/sheet61CC513F/LVDS_IN_P
- R15 pad 1: /LVDS_to_Jetson_lines/VOLT_3P3 -> /LVDS_to_Jetson_lines/Level_shift_and_switch_single/TOP_RDR_HS_D0_N
- R15 pad 2: Net-(R15-Pad2) -> /LVDS_to_Jetson_lines/Level_shift_and_switch_single/sheet61B2E685/sheet61CC513F/LVDS_IN_N
- R16 pad 1: /LVDS_to_Jetson_lines/VOLT_3P3 -> /LVDS_to_Jetson_lines/Level_shift_and_switch_single/TOP_RDR_HS_D0_P
- R16 pad 2: Net-(R16-Pad2) -> Earth
- R17 pad 1: Earth -> /LVDS_to_Jetson_lines/Level_shift_and_switch_single/TOP_RDR_HS_D0_N
- R17 pad 2: /LVDS_to_Jetson_lines/Level_shift_and_switch/sheet61B2E685/DS25_EQ2 -> Earth
- R18 pad 1: Earth -> /LVDS_to_Jetson_lines/Level_shift_and_switch_single/sheet61B2E685/sheet61CC9F81/LVDS_IN_P
- R18 pad 2: /LVDS_to_Jetson_lines/Level_shift_and_switch/sheet61B2E685/DS25_PE1 -> /LVDS_to_Jetson_lines/VOLT_2P5
- R19 pad 1: Earth -> /LVDS_to_Jetson_lines/VOLT_2P5
- R19 pad 2: /LVDS_to_Jetson_lines/Level_shift_and_switch/sheet61B8C8AB/DS25_EQ2 -> /LVDS_to_Jetson_lines/Level_shift_and_switch_single/sheet61B2E685/sheet61CC9F81/LVDS_IN_N
- R20 pad 1: Earth -> /LVDS_to_Jetson_lines/Level_shift_and_switch_single/TOP_RDR_HS_CLK_P
- R20 pad 2: /LVDS_to_Jetson_lines/Level_shift_and_switch/sheet61B8C8AB/DS25_PE1 -> /LVDS_to_Jetson_lines/Level_shift_and_switch_single/sheet61B2E685/sheet61CC9F81/LVDS_IN_P
- R27 pad 1: /LVDS_to_Jetson_lines/Level_shift_and_switch/sheet61B2E685/sheet61CC513F/LVDS_IN_P -> /LVDS_to_Jetson_lines/Level_shift_and_switch_single/TOP_RDR_HS_D1_N
- R27 pad 2: /LVDS_to_Jetson_lines/Level_shift_and_switch/sheet61B2E685/VOLT_2P5 -> /LVDS_to_Jetson_lines/Level_shift_and_switch_single/sheet61B2E685/sheet61CCEEAC/LVDS_IN_N
- R28 pad 1: /LVDS_to_Jetson_lines/Level_shift_and_switch/sheet61B2E685/sheet61CC513F/LVDS_IN_N -> /LVDS_to_Jetson_lines/Level_shift_and_switch_single/TOP_RDR_HS_D1_P
- R28 pad 2: /LVDS_to_Jetson_lines/Level_shift_and_switch/sheet61B2E685/VOLT_2P5 -> Earth
- R29 pad 1: /LVDS_to_Jetson_lines/Level_shift_and_switch/TOP_RDR_HS_D1_P -> /LVDS_to_Jetson_lines/Level_shift_and_switch_single/TOP_RDR_HS_D1_N
- R29 pad 2: /LVDS_to_Jetson_lines/Level_shift_and_switch/sheet61B2E685/sheet61CC513F/LVDS_IN_P -> Earth
- R3 pad 1: Net-(R3-Pad1) -> Earth
- R3 pad 2: /LVDS_to_Jetson_lines/VOLT_3P3 -> /LVDS_to_Jetson_lines/Level_shift_and_switch_single/sheet61B2E685/DS25_EQ2
- R30 pad 1: /LVDS_to_Jetson_lines/Level_shift_and_switch/TOP_RDR_HS_D1_N -> /LVDS_to_Jetson_lines/Level_shift_and_switch_single/sheet61CEF8CC/LVDS_IN_P
- R30 pad 2: /LVDS_to_Jetson_lines/Level_shift_and_switch/sheet61B2E685/sheet61CC513F/LVDS_IN_N -> /LVDS_to_Jetson_lines/VOLT_2P5
- R31 pad 1: /LVDS_to_Jetson_lines/Level_shift_and_switch/TOP_RDR_HS_D1_P -> /LVDS_to_Jetson_lines/VOLT_2P5
- R31 pad 2: Earth -> /LVDS_to_Jetson_lines/Level_shift_and_switch_single/sheet61CEF8CC/LVDS_IN_N
- R32 pad 1: /LVDS_to_Jetson_lines/Level_shift_and_switch/TOP_RDR_HS_D1_N -> /LVDS_to_Jetson_lines/Level_shift_and_switch_single/sheet61CEF8CC/SLVS_OUT_P
- R32 pad 2: Earth -> /LVDS_to_Jetson_lines/Level_shift_and_switch_single/sheet61CEF8CC/LVDS_IN_P
- R33 pad 1: /LVDS_to_Jetson_lines/Level_shift_and_switch/sheet61B2E685/sheet61CC9F81/LVDS_IN_P -> /LVDS_to_Jetson_lines/Level_shift_and_switch_single/sheet61CEF8CC/SLVS_OUT_N
- R33 pad 2: /LVDS_to_Jetson_lines/Level_shift_and_switch/sheet61B2E685/VOLT_2P5 -> /LVDS_to_Jetson_lines/Level_shift_and_switch_single/sheet61CEF8CC/LVDS_IN_N
- R34 pad 1: /LVDS_to_Jetson_lines/Level_shift_and_switch/sheet61B2E685/sheet61CC9F81/LVDS_IN_N -> Earth
- R34 pad 2: /LVDS_to_Jetson_lines/Level_shift_and_switch/sheet61B2E685/VOLT_2P5 -> /LVDS_to_Jetson_lines/Level_shift_and_switch_single/sheet61CEF8CC/SLVS_OUT_P
- R35 pad 1: /LVDS_to_Jetson_lines/Level_shift_and_switch/TOP_RDR_HS_D0_P -> /LVDS_to_Jetson_lines/Level_shift_and_switch_single/sheet61CEF8CC/SLVS_OUT_N
- R35 pad 2: /LVDS_to_Jetson_lines/Level_shift_and_switch/sheet61B2E685/sheet61CC9F81/LVDS_IN_P -> Earth
- R36 pad 1: /LVDS_to_Jetson_lines/Level_shift_and_switch/TOP_RDR_HS_D0_N -> /LVDS_to_Jetson_lines/Level_shift_and_switch_single/sheet61CEF8CC/SLVS_OUT_N
- R36 pad 2: /LVDS_to_Jetson_lines/Level_shift_and_switch/sheet61B2E685/sheet61CC9F81/LVDS_IN_N -> /LVDS_to_Jetson_lines/Level_shift_and_switch_single/sheet61CEF8CC/SLVS_OUT_P
- R37 pad 1: /LVDS_to_Jetson_lines/Level_shift_and_switch/TOP_RDR_HS_D0_P -> /LVDS_to_Jetson_lines/LVDS_to_Jetson_simple/LVDS_2_SLVS_experimental/LVDS_IN_P
- R37 pad 2: Earth -> /LVDS_to_Jetson_lines/VOLT_2P5
- R38 pad 1: /LVDS_to_Jetson_lines/Level_shift_and_switch/TOP_RDR_HS_D0_N -> /LVDS_to_Jetson_lines/VOLT_2P5
- R38 pad 2: Earth -> /LVDS_to_Jetson_lines/LVDS_to_Jetson_simple/LVDS_2_SLVS_experimental/LVDS_IN_N
- R39 pad 1: /LVDS_to_Jetson_lines/Level_shift_and_switch/sheet61B2E685/sheet61CCEEAC/LVDS_IN_P -> /LVDS_to_Jetson_lines/LVDS_to_Jetson_simple/EXP_HS_D1_P
- R39 pad 2: /LVDS_to_Jetson_lines/Level_shift_and_switch/sheet61B2E685/VOLT_2P5 -> /LVDS_to_Jetson_lines/LVDS_to_Jetson_simple/LVDS_2_SLVS_experimental/LVDS_IN_P
- R4 pad 1: Net-(R4-Pad1) -> Earth
- R4 pad 2: /LVDS_to_Jetson_lines/VOLT_3P3 -> /LVDS_to_Jetson_lines/Level_shift_and_switch_single/sheet61B2E685/DS25_PE1
- R40 pad 1: /LVDS_to_Jetson_lines/Level_shift_and_switch/sheet61B2E685/sheet61CCEEAC/LVDS_IN_N -> /LVDS_to_Jetson_lines/LVDS_to_Jetson_simple/EXP_HS_D1_N
- R40 pad 2: /LVDS_to_Jetson_lines/Level_shift_and_switch/sheet61B2E685/VOLT_2P5 -> /LVDS_to_Jetson_lines/LVDS_to_Jetson_simple/LVDS_2_SLVS_experimental/LVDS_IN_N
- R41 pad 1: /LVDS_to_Jetson_lines/Level_shift_and_switch/TOP_RDR_HS_CLK_P -> Earth
- R41 pad 2: /LVDS_to_Jetson_lines/Level_shift_and_switch/sheet61B2E685/sheet61CCEEAC/LVDS_IN_P -> /LVDS_to_Jetson_lines/LVDS_to_Jetson_simple/EXP_HS_D1_P
- R42 pad 1: /LVDS_to_Jetson_lines/Level_shift_and_switch/TOP_RDR_HS_CLK_N -> /LVDS_to_Jetson_lines/LVDS_to_Jetson_simple/EXP_HS_D1_N
- R42 pad 2: /LVDS_to_Jetson_lines/Level_shift_and_switch/sheet61B2E685/sheet61CCEEAC/LVDS_IN_N -> Earth
- R43 pad 1: /LVDS_to_Jetson_lines/Level_shift_and_switch/TOP_RDR_HS_CLK_P -> /LVDS_to_Jetson_lines/LVDS_to_Jetson_simple/EXP_TST_SWITCHED_P
- R43 pad 2: Earth -> /LVDS_to_Jetson_lines/LVDS_to_Jetson_simple/EXP_TST_SWITCHED_N
- R44 pad 1: /LVDS_to_Jetson_lines/Level_shift_and_switch/TOP_RDR_HS_CLK_N -> /LVDS_to_Jetson_lines/LVDS_to_Jetson_simple/sheet61DCF818/LVDS_IN_P
- R44 pad 2: Earth -> /LVDS_to_Jetson_lines/VOLT_2P5
- R5 pad 2: /LVDS_to_Jetson_lines/Level_shift_and_switch/sheet61B2E685/DS25_EQ0 -> /LVDS_to_Jetson_lines/Level_shift_and_switch_single/sheet61B2E685/DS25_EQ0
- R51 pad 1: /LVDS_to_Jetson_lines/Level_shift_and_switch/sheet61B8C8AB/sheet61CC513F/LVDS_IN_P -> /LVDS_to_Jetson_lines/VOLT_2P5
- R51 pad 2: /LVDS_to_Jetson_lines/Level_shift_and_switch/sheet61B8C8AB/VOLT_2P5 -> /LVDS_to_Jetson_lines/LVDS_to_Jetson_simple/sheet61E06ACF/LVDS_IN_N
- R52 pad 1: /LVDS_to_Jetson_lines/Level_shift_and_switch/sheet61B8C8AB/sheet61CC513F/LVDS_IN_N -> /LVDS_to_Jetson_lines/LVDS_to_Jetson_simple/EXP_HS_CLK_P
- R52 pad 2: /LVDS_to_Jetson_lines/Level_shift_and_switch/sheet61B8C8AB/VOLT_2P5 -> /LVDS_to_Jetson_lines/LVDS_to_Jetson_simple/sheet61E06ACF/LVDS_IN_P
- R53 pad 1: /LVDS_to_Jetson_lines/Level_shift_and_switch/BOT_RDR_HS_CLK_P -> /LVDS_to_Jetson_lines/LVDS_to_Jetson_simple/EXP_HS_CLK_N
- R53 pad 2: /LVDS_to_Jetson_lines/Level_shift_and_switch/sheet61B8C8AB/sheet61CC513F/LVDS_IN_P -> /LVDS_to_Jetson_lines/LVDS_to_Jetson_simple/sheet61E06ACF/LVDS_IN_N
- R54 pad 1: /LVDS_to_Jetson_lines/Level_shift_and_switch/BOT_RDR_HS_CLK_N -> Earth
- R54 pad 2: /LVDS_to_Jetson_lines/Level_shift_and_switch/sheet61B8C8AB/sheet61CC513F/LVDS_IN_N -> /LVDS_to_Jetson_lines/LVDS_to_Jetson_simple/EXP_HS_CLK_P
- R55 pad 1: /LVDS_to_Jetson_lines/Level_shift_and_switch/BOT_RDR_HS_CLK_P -> /LVDS_to_Jetson_lines/LVDS_to_Jetson_simple/EXP_HS_CLK_N
- R56 pad 1: /LVDS_to_Jetson_lines/Level_shift_and_switch/BOT_RDR_HS_CLK_N -> /LVDS_to_Jetson_lines/LVDS_to_Jetson_simple/sheet61E220DB/LVDS_IN_P
- R56 pad 2: Earth -> /LVDS_to_Jetson_lines/VOLT_2P5
- R57 pad 1: /LVDS_to_Jetson_lines/Level_shift_and_switch/sheet61B8C8AB/sheet61CC9F81/LVDS_IN_P -> /LVDS_to_Jetson_lines/VOLT_2P5
- R57 pad 2: /LVDS_to_Jetson_lines/Level_shift_and_switch/sheet61B8C8AB/VOLT_2P5 -> /LVDS_to_Jetson_lines/LVDS_to_Jetson_simple/sheet61E220DB/LVDS_IN_N
- R58 pad 1: /LVDS_to_Jetson_lines/Level_shift_and_switch/sheet61B8C8AB/sheet61CC9F81/LVDS_IN_N -> /LVDS_to_Jetson_lines/LVDS_to_Jetson_simple/EXP_HS_D0_P
- R58 pad 2: /LVDS_to_Jetson_lines/Level_shift_and_switch/sheet61B8C8AB/VOLT_2P5 -> /LVDS_to_Jetson_lines/LVDS_to_Jetson_simple/sheet61E220DB/LVDS_IN_P
- R59 pad 1: /LVDS_to_Jetson_lines/Level_shift_and_switch/BOT_RDR_HS_D0_P -> /LVDS_to_Jetson_lines/LVDS_to_Jetson_simple/EXP_HS_D0_N
- R59 pad 2: /LVDS_to_Jetson_lines/Level_shift_and_switch/sheet61B8C8AB/sheet61CC9F81/LVDS_IN_P -> /LVDS_to_Jetson_lines/LVDS_to_Jetson_simple/sheet61E220DB/LVDS_IN_N
- R6 pad 2: /LVDS_to_Jetson_lines/Level_shift_and_switch/sheet61B2E685/DS25_PE0 -> /LVDS_to_Jetson_lines/Level_shift_and_switch_single/sheet61B2E685/DS25_PE0
- R60 pad 1: /LVDS_to_Jetson_lines/Level_shift_and_switch/BOT_RDR_HS_D0_N -> Earth
- R60 pad 2: /LVDS_to_Jetson_lines/Level_shift_and_switch/sheet61B8C8AB/sheet61CC9F81/LVDS_IN_N -> /LVDS_to_Jetson_lines/LVDS_to_Jetson_simple/EXP_HS_D0_P
- R61 pad 1: /LVDS_to_Jetson_lines/Level_shift_and_switch/BOT_RDR_HS_D0_P -> /LVDS_to_Jetson_lines/LVDS_to_Jetson_simple/EXP_HS_D0_N
- R7 pad 1: /LVDS_to_Jetson_lines/VOLT_3P3 -> Net-(R7-Pad1)
- R7 pad 2: Net-(R7-Pad2) -> /LVDS_to_Jetson_lines/VOLT_3P3
- R8 pad 1: /LVDS_to_Jetson_lines/VOLT_3P3 -> Net-(R8-Pad1)
- R8 pad 2: Net-(R8-Pad2) -> /LVDS_to_Jetson_lines/VOLT_3P3
- U1 pad 11: Earth -> (no net)
- U1 pad 26: /LVDS_to_Jetson_lines/Level_shift_and_switch/TOP_1P2_LP_D1_P -> /LVDS_to_Jetson_lines/Level_shift_and_switch_single/TOP_1P2_LP_D0_P
- U1 pad 27: /LVDS_to_Jetson_lines/Level_shift_and_switch/TOP_1P2_LP_D1_N -> /LVDS_to_Jetson_lines/Level_shift_and_switch_single/TOP_1P2_LP_D0_N
- U1 pad 29: /LVDS_to_Jetson_lines/Level_shift_and_switch/TOP_1P2_LP_D0_P -> /LVDS_to_Jetson_lines/Level_shift_and_switch_single/TOP_1P2_LP_CLK_P
- U1 pad 30: /LVDS_to_Jetson_lines/Level_shift_and_switch/TOP_1P2_LP_D0_N -> /LVDS_to_Jetson_lines/Level_shift_and_switch_single/TOP_1P2_LP_CLK_N
- U1 pad 32: /LVDS_to_Jetson_lines/Level_shift_and_switch/TOP_1P2_LP_CLK_P -> (no net)
- U1 pad 33: /LVDS_to_Jetson_lines/Level_shift_and_switch/TOP_1P2_LP_CLK_N -> (no net)
- U1 pad 38: Earth -> /LVDS_to_Jetson_lines/Level_shift_and_switch_single/TOP_1P2_LP_D1_P
- U1 pad 40: /LVDS_to_Jetson_lines/Level_shift_and_switch/BOT_1P2_LP_CLK_P -> (no net)
- U1 pad 43: /LVDS_to_Jetson_lines/Level_shift_and_switch/BOT_1P2_LP_D0_P -> (no net)
- U1 pad 44: /LVDS_to_Jetson_lines/Level_shift_and_switch/BOT_1P2_LP_D0_N -> (no net)
- U1 pad 46: /LVDS_to_Jetson_lines/Level_shift_and_switch/BOT_1P2_LP_D1_P -> (no net)
- U1 pad 47: /LVDS_to_Jetson_lines/Level_shift_and_switch/BOT_1P2_LP_D1_N -> (no net)
- U2 pad 15: CSI_C_D1_N -> (no net)
- U2 pad 16: CSI_C_D1_P -> (no net)
- U2 pad 18: /LVDS_to_Jetson_lines/Level_shift_and_switch/TOP_1P2_LP_D1_P -> (no net)
- U2 pad 19: /LVDS_to_Jetson_lines/Level_shift_and_switch/TOP_RDR_HS_D1_P -> (no net)
- U2 pad 2: CSI_D_D1_N -> (no net)
- U2 pad 20: /LVDS_to_Jetson_lines/Level_shift_and_switch/TOP_1P2_LP_D1_N -> (no net)
- U2 pad 21: /LVDS_to_Jetson_lines/Level_shift_and_switch/TOP_RDR_HS_D1_N -> (no net)
- U2 pad 22: /LVDS_to_Jetson_lines/Level_shift_and_switch/TOP_1P2_LP_D0_P -> /LVDS_to_Jetson_lines/Level_shift_and_switch_single/TOP_1P2_LP_D0_P
- U2 pad 23: /LVDS_to_Jetson_lines/Level_shift_and_switch/TOP_RDR_HS_D0_P -> /LVDS_to_Jetson_lines/Level_shift_and_switch_single/TOP_RDR_HS_D0_P
- U2 pad 24: /LVDS_to_Jetson_lines/Level_shift_and_switch/TOP_1P2_LP_D0_N -> /LVDS_to_Jetson_lines/Level_shift_and_switch_single/TOP_1P2_LP_D0_N
- U2 pad 25: /LVDS_to_Jetson_lines/Level_shift_and_switch/TOP_RDR_HS_D0_N -> /LVDS_to_Jetson_lines/Level_shift_and_switch_single/TOP_RDR_HS_D0_N
- U2 pad 26: /LVDS_to_Jetson_lines/Level_shift_and_switch/TOP_1P2_LP_CLK_P -> /LVDS_to_Jetson_lines/Level_shift_and_switch_single/TOP_1P2_LP_CLK_P
- U2 pad 27: /LVDS_to_Jetson_lines/Level_shift_and_switch/TOP_RDR_HS_CLK_P -> /LVDS_to_Jetson_lines/Level_shift_and_switch_single/TOP_RDR_HS_CLK_P
- U2 pad 28: /LVDS_to_Jetson_lines/Level_shift_and_switch/TOP_1P2_LP_CLK_N -> /LVDS_to_Jetson_lines/Level_shift_and_switch_single/TOP_1P2_LP_CLK_N
- U2 pad 29: /LVDS_to_Jetson_lines/Level_shift_and_switch/TOP_RDR_HS_CLK_N -> /LVDS_to_Jetson_lines/Level_shift_and_switch_single/TOP_RDR_HS_CLK_N
- U2 pad 3: CSI_D_D1_P -> (no net)
- U2 pad 31: /LVDS_to_Jetson_lines/Level_shift_and_switch/BOT_1P2_LP_CLK_P -> /LVDS_to_Jetson_lines/Level_shift_and_switch_single/TOP_1P2_LP_D1_P
- U2 pad 32: /LVDS_to_Jetson_lines/Level_shift_and_switch/BOT_RDR_HS_CLK_P -> /LVDS_to_Jetson_lines/Level_shift_and_switch_single/TOP_RDR_HS_D1_P
- U2 pad 34: /LVDS_to_Jetson_lines/Level_shift_and_switch/BOT_RDR_HS_CLK_N -> /LVDS_to_Jetson_lines/Level_shift_and_switch_single/TOP_RDR_HS_D1_N
- U2 pad 35: /LVDS_to_Jetson_lines/Level_shift_and_switch/BOT_1P2_LP_D0_P -> (no net)
- U2 pad 36: /LVDS_to_Jetson_lines/Level_shift_and_switch/BOT_RDR_HS_D0_P -> (no net)
- U2 pad 37: /LVDS_to_Jetson_lines/Level_shift_and_switch/BOT_1P2_LP_D0_N -> (no net)
- U2 pad 38: /LVDS_to_Jetson_lines/Level_shift_and_switch/BOT_RDR_HS_D0_N -> (no net)
- U2 pad 39: /LVDS_to_Jetson_lines/Level_shift_and_switch/BOT_RDR_HS_D1_P -> (no net)
- U2 pad 4: CSI_D_D0_N -> (no net)
- U2 pad 40: /LVDS_to_Jetson_lines/Level_shift_and_switch/BOT_1P2_LP_D1_P -> (no net)
- U2 pad 41: /LVDS_to_Jetson_lines/Level_shift_and_switch/BOT_RDR_HS_D1_N -> (no net)
- U2 pad 42: /LVDS_to_Jetson_lines/Level_shift_and_switch/BOT_1P2_LP_D1_N -> (no net)
- U2 pad 5: CSI_D_D0_P -> (no net)
- U2 pad 6: CSI_D_CLK_N -> CSI_C_D1_N
- U2 pad 7: CSI_D_CLK_P -> CSI_C_D1_P
- U3 pad 3: /LVDS_to_Jetson_lines/VOLT_3P3 -> Earth
- U3 pad 4: (no net) -> /LVDS_to_Jetson_lines/Level_shift_and_switch_single/SWITCH_HS_0_LP_1_3V3
- U3 pad 5: (no net) -> /LVDS_to_Jetson_lines/VOLT_3P3
- U4 pad 11: /LVDS_to_Jetson_lines/Level_shift_and_switch/sheet61B8C8AB/DS25_EQ2 -> /LVDS_to_Jetson_lines/Level_shift_and_switch_single/sheet61B2E685/DS25_EQ2
- U4 pad 12: /LVDS_to_Jetson_lines/Level_shift_and_switch/sheet61B8C8AB/DS25_EQ2 -> /LVDS_to_Jetson_lines/Level_shift_and_switch_single/sheet61B2E685/DS25_EQ2
- U4 pad 13: Net-(R10-Pad1) -> Net-(R7-Pad1)
- U4 pad 14: Net-(R11-Pad1) -> Net-(R8-Pad1)
- U4 pad 18: /LVDS_to_Jetson_lines/Level_shift_and_switch/sheet61B8C8AB/DS25_PE1 -> /LVDS_to_Jetson_lines/Level_shift_and_switch_single/sheet61B2E685/DS25_PE1
- U4 pad 19: /LVDS_to_Jetson_lines/Level_shift_and_switch/sheet61B8C8AB/DS25_PE1 -> /LVDS_to_Jetson_lines/Level_shift_and_switch_single/sheet61B2E685/DS25_PE1
- U4 pad 20: /LVDS_to_Jetson_lines/Level_shift_and_switch/sheet61B8C8AB/DS25_PE1 -> /LVDS_to_Jetson_lines/Level_shift_and_switch_single/sheet61B2E685/DS25_PE1
- U4 pad 21: /LVDS_to_Jetson_lines/Level_shift_and_switch/sheet61B8C8AB/sheet61CCEEAC/LVDS_IN_N -> /LVDS_to_Jetson_lines/Level_shift_and_switch_single/sheet61B2E685/sheet61CCEEAC/LVDS_IN_N
- U4 pad 22: /LVDS_to_Jetson_lines/Level_shift_and_switch/sheet61B8C8AB/sheet61CCEEAC/LVDS_IN_P -> /LVDS_to_Jetson_lines/Level_shift_and_switch_single/sheet61B2E685/sheet61CCEEAC/LVDS_IN_P
- U4 pad 23: /LVDS_to_Jetson_lines/Level_shift_and_switch/sheet61B8C8AB/sheet61CC9F81/LVDS_IN_N -> /LVDS_to_Jetson_lines/Level_shift_and_switch_single/sheet61B2E685/sheet61CC9F81/LVDS_IN_N
- U4 pad 24: /LVDS_to_Jetson_lines/Level_shift_and_switch/sheet61B8C8AB/sheet61CC9F81/LVDS_IN_P -> /LVDS_to_Jetson_lines/Level_shift_and_switch_single/sheet61B2E685/sheet61CC9F81/LVDS_IN_P
- U4 pad 26: /LVDS_to_Jetson_lines/Level_shift_and_switch/sheet61B8C8AB/sheet61CC513F/LVDS_IN_N -> /LVDS_to_Jetson_lines/Level_shift_and_switch_single/sheet61B2E685/sheet61CC513F/LVDS_IN_N
- U4 pad 27: /LVDS_to_Jetson_lines/Level_shift_and_switch/sheet61B8C8AB/sheet61CC513F/LVDS_IN_P -> /LVDS_to_Jetson_lines/Level_shift_and_switch_single/sheet61B2E685/sheet61CC513F/LVDS_IN_P
- U4 pad 28: (no net) -> /LVDS_to_Jetson_lines/Level_shift_and_switch_single/sheet61CEF8CC/LVDS_IN_N
- U4 pad 29: (no net) -> /LVDS_to_Jetson_lines/Level_shift_and_switch_single/sheet61CEF8CC/LVDS_IN_P
- U4 pad 31: /LVDS_to_Jetson_lines/Level_shift_and_switch/sheet61B8C8AB/DS25_PE0 -> /LVDS_to_Jetson_lines/Level_shift_and_switch_single/sheet61B2E685/DS25_PE0
- U4 pad 32: Net-(R15-Pad2) -> Net-(R10-Pad2)
- U4 pad 33: Net-(R15-Pad2) -> Net-(R10-Pad2)
- U4 pad 34: Net-(R15-Pad2) -> Net-(R10-Pad2)
- U4 pad 35: Net-(R15-Pad2) -> Net-(R10-Pad2)
- U4 pad 36: Net-(R16-Pad2) -> Net-(R11-Pad2)
- U4 pad 37: Net-(R14-Pad2) -> Net-(R9-Pad2)
- U4 pad 38: Net-(R15-Pad2) -> Net-(R10-Pad2)
- U4 pad 39: /LVDS_to_Jetson_lines/Level_shift_and_switch/sheet61B8C8AB/DS25_EQ0 -> /LVDS_to_Jetson_lines/Level_shift_and_switch_single/sheet61B2E685/DS25_EQ0
- U4 pad 40: /LVDS_to_Jetson_lines/Level_shift_and_switch/sheet61B8C8AB/DS25_EQ0 -> /LVDS_to_Jetson_lines/Level_shift_and_switch_single/sheet61B2E685/DS25_EQ0
- U5 pad 3: Earth -> (no net)
- U5 pad 4: /LVDS_to_Jetson_lines/Level_shift_and_switch/SWITCH_HS_0_LP_1_3V3 -> CSI_A_D1_N
- U5 pad 5: /LVDS_to_Jetson_lines/VOLT_3P3 -> CSI_A_D1_P
Other:
- board text added: "NOTE: Place all components at grid spacing of 20 mils!!!"

Commit message: rev 2022
Parts:
- added C14: 0.1uF, Capacitors_SMD:C_0402, B.Cu at (146.7, 72.6)
- added C15: 0.1uF, Capacitors_SMD:C_0402, B.Cu at (151.0, 72.6)
- added C16: 0.1uF, Capacitors_SMD:C_0402, B.Cu at (146.6, 84.2)
- added C17: 0.1uF, Capacitors_SMD:C_0402, B.Cu at (151.1, 84.3)
- added C18: 0.1uF, Capacitors_SMD:C_0402, F.Cu at (142.5, 94.1)
- added C19: 0.1uF, Capacitors_SMD:C_0402, F.Cu at (134.2, 98.1)
- added C20: 0.1uF, Capacitors_SMD:C_0402, F.Cu at (140.0, 104.4)
- added C21: 0.1uF, Capacitors_SMD:C_0402, F.Cu at (134.3, 112.8)
- added C22: 0.1uF, Capacitors_SMD:C_0402, F.Cu at (140.0, 106.8)
- added C23: 0.1uF, Capacitors_SMD:C_0402, F.Cu at (140.9, 118.4)
- added R62: 9.1, Resistors_SMD:R_0603_HandSoldering, F.Cu at (110.1, 62.8)
- added R63: 220, Resistors_SMD:R_0603, F.Cu at (109.8, 128.8)
- added R64: 220, Resistors_SMD:R_0603, F.Cu at (109.8, 125.5)
- added R65: 47, Resistors_SMD:R_0603, F.Cu at (112.5, 128.2)
- added R66: 47, Resistors_SMD:R_0603, F.Cu at (112.5, 126.0)
- added R67: 9.1, Resistors_SMD:R_0603_HandSoldering, F.Cu at (115.3, 129.5)
- added R68: 9.1, Resistors_SMD:R_0603_HandSoldering, F.Cu at (115.3, 124.8)
- added R69: 220, Resistors_SMD:R_0603, F.Cu at (114.2, 118.6)
- added R70: 220, Resistors_SMD:R_0603, F.Cu at (114.3, 115.0)
- added R71: 47, Resistors_SMD:R_0603, F.Cu at (117.2, 118.1)
- added R72: 47, Resistors_SMD:R_0603, F.Cu at (117.0, 115.6)
- added R73: 9.1, Resistors_SMD:R_0603_HandSoldering, F.Cu at (120.2, 119.2)
- added R74: 9.1, Resistors_SMD:R_0603_HandSoldering, F.Cu at (120.2, 114.3)
- added U6: TS3DDR3812_RUA_42, FMC_MIPI_v2_sym:TS3DDR3812RUAR, F.Cu at (138.7, 112.8)
- added U8: SN74AVCH16T245_DGV_48, FMC_MIPI_v2_sym:DGV48, B.Cu at (148.9, 78.9)
- R16, R17, R22, R23, R28, R29: value 12 -> 9.1; footprint Resistors_SMD:R_0805 -> Resistors_SMD:R_0603_HandSoldering
- R37, R38: value 220 -> 0; footprint Resistors_SMD:R_0603 -> Resistors_SMD:R_0805
- R39, R40, R46, R52, R58: value 47 -> 220
- R41, R42, R48, R54, R60: value 10 -> 47; footprint Resistors_SMD:R_1206_HandSoldering -> Resistors_SMD:R_0603
- R43: value 100 -> 9.1; footprint Resistors_SMD:R_1206_HandSoldering -> Resistors_SMD:R_0603_HandSoldering
- R44, R50, R56: value 220 -> 9.1; footprint Resistors_SMD:R_0603 -> Resistors_SMD:R_0603_HandSoldering
- R49, R55, R61: value 10 -> 9.1; footprint Resistors_SMD:R_1206_HandSoldering -> Resistors_SMD:R_0603_HandSoldering
- moved U2 212.3 mm to (-64.8, 30.9)
- moved R44 168.6 mm to (114.1, 100.2), turned to 270 degrees
- moved R37 167.4 mm to (134.1, 92.1), turned to 180 degrees
- moved R38 167.2 mm to (134.2, 105.4), turned to 180 degrees
- moved R47 167.0 mm to (115.9, 93.1)
- moved R45 166.8 mm to (113.1, 93.7)
- moved R49 166.7 mm to (118.7, 94.3)
- moved R50 165.6 mm to (118.8, 89.3), turned to 270 degrees
- moved R46 164.1 mm to (113.1, 90.2), turned to 270 degrees
- moved R48 164.0 mm to (115.8, 90.7), turned to 180 degrees
- moved R53 160.9 mm to (115.8, 79.6)
- moved R51 160.6 mm to (113.0, 80.1), turned to 270 degrees
- moved R55 160.5 mm to (118.8, 80.8)
- moved R52 158.2 mm to (113.1, 76.6), turned to 270 degrees
- moved R54 157.1 mm to (115.8, 77.2), turned to 180 degrees
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Connections:
- J2 pad 1: CSI_A_D0_P -> (no net)
- J2 pad 13: CSI_A_D1_P -> (no net)
- J2 pad 15: CSI_A_D1_N -> (no net)
- J2 pad 20: (no net) -> CSI_D_D0_P
- J2 pad 22: (no net) -> CSI_D_D0_N
- J2 pad 26: (no net) -> CSI_D_CLK_P
- J2 pad 28: (no net) -> CSI_D_CLK_N
- J2 pad 3: CSI_A_D0_N -> (no net)
- J2 pad 32: (no net) -> CSI_D_D1_P
- J2 pad 34: (no net) -> CSI_D_D1_N
- J2 pad 7: CSI_A_CLK_P -> (no net)
- J2 pad 9: CSI_A_CLK_N -> (no net)
- R17 pad 1: /LVDS_to_Jetson_lines/Level_shift_and_switch_single/TOP_RDR_HS_D0_N -> Earth
- R17 pad 2: Earth -> /LVDS_to_Jetson_lines/Level_shift_and_switch_single/TOP_RDR_HS_D0_N
- R23 pad 1: /LVDS_to_Jetson_lines/Level_shift_and_switch_single/TOP_RDR_HS_CLK_N -> Earth
- R23 pad 2: Earth -> /LVDS_to_Jetson_lines/Level_shift_and_switch_single/TOP_RDR_HS_CLK_N
- R29 pad 1: /LVDS_to_Jetson_lines/Level_shift_and_switch_single/TOP_RDR_HS_D1_N -> Earth
- R29 pad 2: Earth -> /LVDS_to_Jetson_lines/Level_shift_and_switch_single/TOP_RDR_HS_D1_N
- R37 pad 1: /LVDS_to_Jetson_lines/LVDS_to_Jetson_simple/LVDS_2_SLVS_experimental/LVDS_IN_P -> /LVDS_to_Jetson_lines/EN
- R37 pad 2: /LVDS_to_Jetson_lines/VOLT_2P5 -> /LVDS_to_Jetson_lines/VOLT_3P3
- R38 pad 1: /LVDS_to_Jetson_lines/VOLT_2P5 -> /LVDS_to_Jetson_lines/EN
- R38 pad 2: /LVDS_to_Jetson_lines/LVDS_to_Jetson_simple/LVDS_2_SLVS_experimental/LVDS_IN_N -> /LVDS_to_Jetson_lines/VOLT_3P3
- R39 pad 1: /LVDS_to_Jetson_lines/LVDS_to_Jetson_simple/EXP_HS_D1_P -> /LVDS_to_Jetson_lines/FMC_HS_CSI_C_D1_N
- R39 pad 2: /LVDS_to_Jetson_lines/LVDS_to_Jetson_simple/LVDS_2_SLVS_experimental/LVDS_IN_P -> /LVDS_to_Jetson_lines/VOLT_2P5
- R40 pad 1: /LVDS_to_Jetson_lines/LVDS_to_Jetson_simple/EXP_HS_D1_N -> /LVDS_to_Jetson_lines/VOLT_2P5
- R40 pad 2: /LVDS_to_Jetson_lines/LVDS_to_Jetson_simple/LVDS_2_SLVS_experimental/LVDS_IN_N -> /LVDS_to_Jetson_lines/FMC_HS_CSI_C_D1_P
- R41 pad 1: Earth -> /LVDS_to_Jetson_lines/HS_CSI_C_D1_N
- R41 pad 2: /LVDS_to_Jetson_lines/LVDS_to_Jetson_simple/EXP_HS_D1_P -> /LVDS_to_Jetson_lines/FMC_HS_CSI_C_D1_N
- R42 pad 1: /LVDS_to_Jetson_lines/LVDS_to_Jetson_simple/EXP_HS_D1_N -> /LVDS_to_Jetson_lines/HS_CSI_C_D1_P
- R42 pad 2: Earth -> /LVDS_to_Jetson_lines/FMC_HS_CSI_C_D1_P
- R43 pad 1: /LVDS_to_Jetson_lines/LVDS_to_Jetson_simple/EXP_TST_SWITCHED_P -> /LVDS_to_Jetson_lines/HS_CSI_C_D1_N
- R43 pad 2: /LVDS_to_Jetson_lines/LVDS_to_Jetson_simple/EXP_TST_SWITCHED_N -> Earth
- R44 pad 1: /LVDS_to_Jetson_lines/LVDS_to_Jetson_simple/sheet61DCF818/LVDS_IN_P -> Earth
- R44 pad 2: /LVDS_to_Jetson_lines/VOLT_2P5 -> /LVDS_to_Jetson_lines/HS_CSI_C_D1_P
- R45 pad 1: /LVDS_to_Jetson_lines/VOLT_2P5 -> /LVDS_to_Jetson_lines/FMC_HS_CSI_C_D0_N
- R45 pad 2: /LVDS_to_Jetson_lines/LVDS_to_Jetson_simple/sheet61DCF818/LVDS_IN_N -> /LVDS_to_Jetson_lines/VOLT_2P5
- R46 pad 1: /LVDS_to_Jetson_lines/LVDS_to_Jetson_simple/EXP_TST_P -> /LVDS_to_Jetson_lines/VOLT_2P5
- R46 pad 2: /LVDS_to_Jetson_lines/LVDS_to_Jetson_simple/sheet61DCF818/LVDS_IN_P -> /LVDS_to_Jetson_lines/FMC_HS_CSI_C_D0_P
- R47 pad 1: /LVDS_to_Jetson_lines/LVDS_to_Jetson_simple/EXP_TST_N -> /LVDS_to_Jetson_lines/HS_CSI_C_D0_N
- R47 pad 2: /LVDS_to_Jetson_lines/LVDS_to_Jetson_simple/sheet61DCF818/LVDS_IN_N -> /LVDS_to_Jetson_lines/FMC_HS_CSI_C_D0_N
- R48 pad 1: Earth -> /LVDS_to_Jetson_lines/HS_CSI_C_D0_P
- R48 pad 2: /LVDS_to_Jetson_lines/LVDS_to_Jetson_simple/EXP_TST_P -> /LVDS_to_Jetson_lines/FMC_HS_CSI_C_D0_P
- R49 pad 1: /LVDS_to_Jetson_lines/LVDS_to_Jetson_simple/EXP_TST_N -> /LVDS_to_Jetson_lines/HS_CSI_C_D0_N
- R50 pad 1: /LVDS_to_Jetson_lines/LVDS_to_Jetson_simple/sheet61E06ACF/LVDS_IN_P -> Earth
- R50 pad 2: /LVDS_to_Jetson_lines/VOLT_2P5 -> /LVDS_to_Jetson_lines/HS_CSI_C_D0_P
- R51 pad 1: /LVDS_to_Jetson_lines/VOLT_2P5 -> /LVDS_to_Jetson_lines/FMC_HS_CSI_D_D1_N
- R51 pad 2: /LVDS_to_Jetson_lines/LVDS_to_Jetson_simple/sheet61E06ACF/LVDS_IN_N -> /LVDS_to_Jetson_lines/VOLT_2P5
- R52 pad 1: /LVDS_to_Jetson_lines/LVDS_to_Jetson_simple/EXP_HS_CLK_P -> /LVDS_to_Jetson_lines/VOLT_2P5
- R52 pad 2: /LVDS_to_Jetson_lines/LVDS_to_Jetson_simple/sheet61E06ACF/LVDS_IN_P -> /LVDS_to_Jetson_lines/FMC_HS_CSI_D_D1_P
- R53 pad 1: /LVDS_to_Jetson_lines/LVDS_to_Jetson_simple/EXP_HS_CLK_N -> /LVDS_to_Jetson_lines/HS_CSI_D_D1_N
- R53 pad 2: /LVDS_to_Jetson_lines/LVDS_to_Jetson_simple/sheet61E06ACF/LVDS_IN_N -> /LVDS_to_Jetson_lines/FMC_HS_CSI_D_D1_N
- R54 pad 1: Earth -> /LVDS_to_Jetson_lines/HS_CSI_D_D1_P
- R54 pad 2: /LVDS_to_Jetson_lines/LVDS_to_Jetson_simple/EXP_HS_CLK_P -> /LVDS_to_Jetson_lines/FMC_HS_CSI_D_D1_P
- R55 pad 1: /LVDS_to_Jetson_lines/LVDS_to_Jetson_simple/EXP_HS_CLK_N -> /LVDS_to_Jetson_lines/HS_CSI_D_D1_N
- R56 pad 1: /LVDS_to_Jetson_lines/LVDS_to_Jetson_simple/sheet61E220DB/LVDS_IN_P -> Earth
- R56 pad 2: /LVDS_to_Jetson_lines/VOLT_2P5 -> /LVDS_to_Jetson_lines/HS_CSI_D_D1_P
- R57 pad 1: /LVDS_to_Jetson_lines/VOLT_2P5 -> /LVDS_to_Jetson_lines/FMC_HS_CSI_D_D0_N
- R57 pad 2: /LVDS_to_Jetson_lines/LVDS_to_Jetson_simple/sheet61E220DB/LVDS_IN_N -> /LVDS_to_Jetson_lines/VOLT_2P5
- R58 pad 1: /LVDS_to_Jetson_lines/LVDS_to_Jetson_simple/EXP_HS_D0_P -> /LVDS_to_Jetson_lines/VOLT_2P5
- R58 pad 2: /LVDS_to_Jetson_lines/LVDS_to_Jetson_simple/sheet61E220DB/LVDS_IN_P -> /LVDS_to_Jetson_lines/FMC_HS_CSI_D_D0_P
- R59 pad 1: /LVDS_to_Jetson_lines/LVDS_to_Jetson_simple/EXP_HS_D0_N -> /LVDS_to_Jetson_lines/HS_CSI_D_D0_N
- R59 pad 2: /LVDS_to_Jetson_lines/LVDS_to_Jetson_simple/sheet61E220DB/LVDS_IN_N -> /LVDS_to_Jetson_lines/FMC_HS_CSI_D_D0_N
- R60 pad 1: Earth -> /LVDS_to_Jetson_lines/HS_CSI_D_D0_P
- R60 pad 2: /LVDS_to_Jetson_lines/LVDS_to_Jetson_simple/EXP_HS_D0_P -> /LVDS_to_Jetson_lines/FMC_HS_CSI_D_D0_P
- R61 pad 1: /LVDS_to_Jetson_lines/LVDS_to_Jetson_simple/EXP_HS_D0_N -> /LVDS_to_Jetson_lines/HS_CSI_D_D0_N
- U2 pad 11: CSI_C_CLK_N -> (no net)
- U2 pad 12: CSI_C_CLK_P -> (no net)
- U2 pad 13: CSI_C_D0_N -> (no net)
- U2 pad 14: CSI_C_D0_P -> (no net)
- U2 pad 6: CSI_C_D1_N -> (no net)
- U2 pad 7: CSI_C_D1_P -> (no net)
- U5 pad 1: (no net) -> /LVDS_to_Jetson_lines/VOLT_3P3
- U5 pad 11: CSI_A_D0_N -> CSI_D_D1_N
- U5 pad 12: CSI_A_D0_P -> CSI_D_D1_P
- U5 pad 13: (no net) -> CSI_D_D0_N
- U5 pad 14: (no net) -> CSI_D_D0_P
- U5 pad 15: /LVDS_to_Jetson_lines/LVDS_to_Jetson_simple/EXP_TST_SWITCHED_N -> (no net)
- U5 pad 16: /LVDS_to_Jetson_lines/LVDS_to_Jetson_simple/EXP_TST_SWITCHED_P -> (no net)
- U5 pad 17: (no net) -> /LVDS_to_Jetson_lines/VOLT_3P3
- U5 pad 19: /LVDS_to_Jetson_lines/LVDS_to_Jetson_simple/EXP_TST_P -> (no net)
- U5 pad 21: /LVDS_to_Jetson_lines/LVDS_to_Jetson_simple/EXP_TST_N -> (no net)
- U5 pad 22: (no net) -> /LVDS_to_Jetson_lines/LP_CSI_D_D0_P
- U5 pad 23: (no net) -> /LVDS_to_Jetson_lines/HS_CSI_D_D0_P
- U5 pad 24: (no net) -> /LVDS_to_Jetson_lines/LP_CSI_D_D0_N
- U5 pad 25: (no net) -> /LVDS_to_Jetson_lines/HS_CSI_D_D0_N
- U5 pad 26: (no net) -> /LVDS_to_Jetson_lines/LP_CSI_D_D1_P
- U5 pad 27: /LVDS_to_Jetson_lines/LVDS_to_Jetson_simple/EXP_HS_D0_P -> /LVDS_to_Jetson_lines/HS_CSI_D_D1_P
- U5 pad 28: (no net) -> /LVDS_to_Jetson_lines/LP_CSI_D_D1_N
- U5 pad 29: /LVDS_to_Jetson_lines/LVDS_to_Jetson_simple/EXP_HS_D0_N -> /LVDS_to_Jetson_lines/HS_CSI_D_D1_N
- U5 pad 30: (no net) -> /LVDS_to_Jetson_lines/VOLT_3P3
- U5 pad 31: (no net) -> /LVDS_to_Jetson_lines/LP_CSI_C_D0_P
- U5 pad 32: /LVDS_to_Jetson_lines/LVDS_to_Jetson_simple/EXP_HS_CLK_P -> /LVDS_to_Jetson_lines/HS_CSI_C_D0_P
- U5 pad 33: (no net) -> /LVDS_to_Jetson_lines/LP_CSI_C_D0_N
- U5 pad 34: /LVDS_to_Jetson_lines/LVDS_to_Jetson_simple/EXP_HS_CLK_N -> /LVDS_to_Jetson_lines/HS_CSI_C_D0_N
- U5 pad 35: (no net) -> /LVDS_to_Jetson_lines/LP_CSI_C_D1_P
- U5 pad 36: /LVDS_to_Jetson_lines/LVDS_to_Jetson_simple/EXP_HS_D1_P -> /LVDS_to_Jetson_lines/HS_CSI_C_D1_P
- U5 pad 37: (no net) -> /LVDS_to_Jetson_lines/LP_CSI_C_D1_N
- U5 pad 38: /LVDS_to_Jetson_lines/LVDS_to_Jetson_simple/EXP_HS_D1_N -> /LVDS_to_Jetson_lines/HS_CSI_C_D1_N
- U5 pad 4: CSI_A_D1_N -> CSI_C_D1_N
- U5 pad 5: CSI_A_D1_P -> CSI_C_D1_P
- U5 pad 6: CSI_A_CLK_N -> CSI_C_D0_N
- U5 pad 7: CSI_A_CLK_P -> CSI_C_D0_P
- U5 pad 8: (no net) -> /LVDS_to_Jetson_lines/EN
Routing:
- net CSI_D_CLK_P: track 0.00 -> 20.9 mm, vias 0 -> 1
- net CSI_D_CLK_N: track 0.00 -> 20.8 mm, vias 0 -> 1
- net CSI_D_D1_N: track 0.00 -> 15.1 mm, vias 0 -> 1
- net CSI_D_D1_P: track 0.00 -> 15.0 mm, vias 0 -> 1
- net CSI_C_CLK_N: track 0.00 -> 14.8 mm, vias 0 -> 1
- net CSI_C_CLK_P: track 0.00 -> 14.7 mm, vias 0 -> 1
- net CSI_D_D0_P: track 0.00 -> 14.4 mm, vias 0 -> 1
- net CSI_D_D0_N: track 0.00 -> 14.4 mm, vias 0 -> 1
- net CSI_C_D1_P: track 0.00 -> 7.77 mm, vias 0 -> 1
- net CSI_C_D1_N: track 0.00 -> 7.52 mm, vias 0 -> 1
- net CSI_C_D0_P: track 0.00 -> 6.82 mm, vias 0 -> 1
- net CSI_C_D0_N: track 0.00 -> 6.72 mm, vias 0 -> 1

Commit message: minor changes
Parts:
- moved R63 74.5 mm to (150.8, 66.6), turned to 180 degrees
- moved R64 73.7 mm to (154.1, 66.6), turned to 180 degrees
- moved R65 70.5 mm to (151.4, 69.4), turned to 90 degrees
- moved R66 70.0 mm to (153.6, 69.4), turned to 90 degrees
- moved R67 67.1 mm to (150.1, 72.1), turned to 180 degrees
- moved R68 65.8 mm to (154.8, 72.1), turned to 180 degrees
- moved R69 56.9 mm to (140.1, 67.9), turned to 180 degrees
- moved R70 55.4 mm to (143.7, 68.0), turned to 180 degrees
- moved R71 52.7 mm to (140.6, 70.9), turned to 90 degrees
- moved R72 51.9 mm to (143.1, 70.7), turned to 90 degrees
- moved R73 49.3 mm to (139.4, 73.9), turned to 180 degrees
- moved R74 47.1 mm to (144.4, 73.9), turned to 180 degrees
- moved C21 34.0 mm to (146.3, 81.0), turned to 270 degrees
- moved R38 31.3 mm to (153.7, 80.9), turned to 90 degrees
- moved C23 30.7 mm to (140.7, 87.7), turned to 90 degrees
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Connections:
- U6 pad 13: CSI_C_CLK_N -> CSI_D_CLK_N
- U6 pad 14: CSI_C_CLK_P -> CSI_D_CLK_P
- U6 pad 22: /LVDS_to_Jetson_lines/LP_CSI_C_CLK_P -> /LVDS_to_Jetson_lines/LP_CSI_D_CLK_P
- U6 pad 23: /LVDS_to_Jetson_lines/HS_CSI_C_CLK_P -> /LVDS_to_Jetson_lines/HS_CSI_D_CLK_P
- U6 pad 24: /LVDS_to_Jetson_lines/LP_CSI_C_CLK_N -> /LVDS_to_Jetson_lines/LP_CSI_D_CLK_N
- U6 pad 25: /LVDS_to_Jetson_lines/HS_CSI_C_CLK_N -> /LVDS_to_Jetson_lines/HS_CSI_D_CLK_N
- U6 pad 31: /LVDS_to_Jetson_lines/LP_CSI_D_CLK_P -> /LVDS_to_Jetson_lines/LP_CSI_C_CLK_P
- U6 pad 32: /LVDS_to_Jetson_lines/HS_CSI_D_CLK_P -> /LVDS_to_Jetson_lines/HS_CSI_C_CLK_P
- U6 pad 33: /LVDS_to_Jetson_lines/LP_CSI_D_CLK_N -> /LVDS_to_Jetson_lines/LP_CSI_C_CLK_N
- U6 pad 34: /LVDS_to_Jetson_lines/HS_CSI_D_CLK_N -> /LVDS_to_Jetson_lines/HS_CSI_C_CLK_N
- U6 pad 6: CSI_D_CLK_N -> CSI_C_CLK_N
- U6 pad 7: CSI_D_CLK_P -> CSI_C_CLK_P
- U8 pad 11: (no net) -> Earth
Routing:
- net CSI_D_D1_P: track 15.0 -> 21.1 mm
- net CSI_D_D1_N: track 15.1 -> 21.1 mm
- net CSI_D_D0_N: track 14.4 -> 19.3 mm
- net CSI_D_D0_P: track 14.4 -> 19.0 mm
- net CSI_C_CLK_N: track 14.8 -> 18.5 mm
- net CSI_C_CLK_P: track 14.7 -> 17.9 mm
- net CSI_D_CLK_N: track 20.8 -> 22.2 mm
- net CSI_D_CLK_P: track 20.9 -> 21.5 mm
Other:
- board text added: "HS Clocks here"
- board text added: "HS Lanes here"
- board text added: "LP lanes here"

Commit message: fixed 3.3 volt level shifter
Parts:
- removed C10, C11, C12, C13, C3, C4, C5, C6, C7: 0.1uF, Capacitors_SMD:C_0402
- removed C8, C9: 1uF, Capacitors_SMD:C_0603
- removed R10, R11, R7, R8, R9: 4.7k, Resistors_SMD:R_0805
- removed R12, R13, R18, R19, R24, R25, R30, R31: 220, Resistors_SMD:R_0603
- removed R14, R15, R20, R21, R26, R27, R32, R33: 47, Resistors_SMD:R_0603
- removed R16, R17, R22, R23, R28, R29: 9.1, Resistors_SMD:R_0603_HandSoldering
- removed R3, R4, R5, R6: 2.2k, Resistors_SMD:R_0805
- removed R34, R35: 10, Resistors_SMD:R_1206_HandSoldering
- removed R36: 100, Resistors_SMD:R_1206_HandSoldering
- removed U1: SN74AVCH16T245_DGV_48, FMC_MIPI_v2_sym:DGV48
- removed U3: SN74LV1T34DBV, TO_SOT_Packages_SMD:SOT-23-5
- removed U4: DS25BR440_RTA_40, FMC_MIPI_v2_sym:DS25BR440_SQA40A
- added R75: 0, Resistors_SMD:R_0805, F.Cu at (140.5, 106.6)
- R1, R2: moved to F.Cu
- U2: value TS3DDR3812_RUA_42 -> SN74AVC2T45DCUR; footprint FMC_MIPI_v2_sym:TS3DDR3812RUAR -> FMC_MIPI_v2_sym:SN74AVC2T45DCUR
- moved R1 236.0 mm to (147.4, 90.7), turned to 0 degrees
- moved C1 213.9 mm to (95.4, 121.8), turned to 90 degrees
- moved C2 212.3 mm to (95.6, 114.1), turned to 270 degrees
- moved R2 195.3 mm to (99.5, 117.9), turned to 90 degrees
- moved U2 183.4 mm to (96.6, 118.0), turned to 90 degrees
Connections:
- C1 pad 1: /LVDS_to_Jetson_lines/VDD_VADJ -> Earth
- C1 pad 2: Earth -> /LVDS_to_Jetson_lines/VDD_VADJ
- C2 pad 1: /LVDS_to_Jetson_lines/VDD_VADJ -> Earth
- C2 pad 2: Earth -> /LVDS_to_Jetson_lines/VOLT_3P3
- R1 pad 1: Net-(R1-Pad1) -> /LVDS_to_Jetson_lines/SWITCH_U6
- R1 pad 2: /LVDS_to_Jetson_lines/Level_shift_and_switch_single/SWITCH_HS_0_LP_1_3V3 -> /LVDS_to_Jetson_lines/SWITCH_CLOCK_LANES_3V3
- R2 pad 1: Net-(R2-Pad1) -> /LVDS_to_Jetson_lines/VDD_VADJ
- R2 pad 2: /LVDS_to_Jetson_lines/VOLT_3P3 -> /LVDS_to_Jetson_lines/DIR
- U2 pad 1: /LVDS_to_Jetson_lines/VOLT_3P3 -> /LVDS_to_Jetson_lines/VDD_VADJ
- U2 pad 4: (no net) -> Earth
- U2 pad 5: (no net) -> /LVDS_to_Jetson_lines/DIR
- U2 pad 6: (no net) -> /LVDS_to_Jetson_lines/SWITCH_CLOCK_LANES_3V3
- U2 pad 7: (no net) -> /LVDS_to_Jetson_lines/SWITCH_DATA_LANES_3V3
- U2 pad 8: Net-(R2-Pad1) -> /LVDS_to_Jetson_lines/VOLT_3P3
- U5 pad 10: (no net) -> /LVDS_to_Jetson_lines/SWITCH_U5
- U5 pad 9: (no net) -> /LVDS_to_Jetson_lines/SWITCH_U5
- U6 pad 10: (no net) -> /LVDS_to_Jetson_lines/SWITCH_U6
- U6 pad 9: (no net) -> /LVDS_to_Jetson_lines/SWITCH_U6
