File: LVDS_to_Jetson_LP_common.sch (KiCad schematic (older format))
At the start: 22 parts, among them U5 TS3DDR3812_RUA_42, U6 TS3DDR3812_RUA_42, U8 SN74AVCH16T245_DGV_48

Commit message: added 4 bit level shifter VADJ to 3.3 volt
Parts:
- gave numbers to parts that had none: 1
