File: LVDS_2_SLVS.sch (KiCad schematic (older format))
At the start: 6 parts

Commit message: placed nicely the components
Parts:
- R16, R17: footprint Resistors_SMD:R_0603_HandSoldering -> Resistors_SMD:R_0603; Part Number (none) -> CR0603-F/-9R10ELF; Power 250 mW -> 100 mW
Changed lines of the file:
@@
 $Descr A4 11693 8268
 encoding utf-8
-Sheet 9 12
+Sheet 5 12
 Title ""
 Date ""
@@
 AR Path="/6366AF3A/63D3885E/5955E861" Ref="R?"  Part="1"
 AR Path="/6366AF3A/63D47A03/5955E861" Ref="R?"  Part="1"
-F 0 "R69" V 2680 1250 50  0000 C CNN
+F 0 "R39" V 2680 1250 50  0000 C CNN
 F 1 "220" V 2600 1250 50  0000 C CNN
 F 2 "Resistors_SMD:R_0603" V 2530 1250 50  0001 C CNN
@@
 AR Path="/6366AF3A/63D3885E/5955F5C4" Ref="R?"  Part="1"
 AR Path="/6366AF3A/63D47A03/5955F5C4" Ref="R?"  Part="1"
-F 0 "R72" V 2980 1700 50  0000 C CNN
+F 0 "R42" V 2980 1700 50  0000 C CNN
 F 1 "47" V 2900 1700 50  0000 C CNN
 F 2 "Resistors_SMD:R_0603" V 2830 1700 50  0001 C CNN
@@
 AR Path="/6366AF3A/63D3885E/61C6D193" Ref="#PWR?"  Part="1"
 AR Path="/6366AF3A/63D47A03/61C6D193" Ref="#PWR?"  Part="1"
-F 0 "#PWR0127" H 3600 2050 50  0001 C CNN
+F 0 "#PWR0117" H 3600 2050 50  0001 C CNN
 F 1 "Earth" H 3600 2150 50  0001 C CNN
 F 2 "" H 3600 2300 50  0000 C CNN
@@
 AR Path="/6366AF3A/63D3885E/61C6D191" Ref="#PWR?"  Part="1"
 AR Path="/6366AF3A/63D47A03/61C6D191" Ref="#PWR?"  Part="1"
-F 0 "#PWR0128" H 3600 900 50  0001 C CNN
+F 0 "#PWR0118" H 3600 900 50  0001 C CNN
 F 1 "Earth" H 3600 1000 50  0001 C CNN
 F 2 "" H 3600 1150 50  0000 C CNN
@@
 AR Path="/6366AF3A/63D3885E/61C6D194" Ref="R?"  Part="1"
 AR Path="/6366AF3A/63D47A03/61C6D194" Ref="R?"  Part="1"
-F 0 "R70" V 2680 1950 50  0000 C CNN
+F 0 "R40" V 2680 1950 50  0000 C CNN
 F 1 "220" V 2600 1950 50  0000 C CNN
 F 2 "Resistors_SMD:R_0603" V 2530 1950 50  0001 C CNN
@@
 AR Path="/6366AF3A/63D3885E/61C6D195" Ref="R?"  Part="1"
 AR Path="/6366AF3A/63D47A03/61C6D195" Ref="R?"  Part="1"
-F 0 "R71" V 2980 1500 50  0000 C CNN
+F 0 "R41" V 2980 1500 50  0000 C CNN
 F 1 "47" V 2900 1500 50  0000 C CNN
 F 2 "Resistors_SMD:R_0603" V 2830 1500 50  0001 C CNN
@@
 AR Path="/6366AF3A/63D3885E/5955E920" Ref="R?"  Part="1"
 AR Path="/6366AF3A/63D47A03/5955E920" Ref="R?"  Part="1"
-F 0 "R73" V 3430 1250 50  0000 C CNN
+F 0 "R43" V 3430 1250 50  0000 C CNN
 F 1 "9.1" V 3350 1250 50  0000 C CNN
-F 2 "Resistors_SMD:R_0603_HandSoldering" V 3280 1250 50  0001 C CNN
-F 3 "" H 3350 1250 50  0001 C CNN
+F 2 "Resistors_SMD:R_0603" V 3280 1250 50  0001 C CNN
+F 3 "https://www.mouser.co.il/ProductDetail/Bourns/CR0603-F-9R10ELF?qs=W%2FMpXkg%252BdQ6lipKjUosapQ%3D%3D" H 3350 1250 50  0001 C CNN
 F 4 "1%" V 3350 1250 60  0001 C CNN "Tolerance"
-F 5 "250 mW" V 3350 1250 60  0001 C CNN "Power"
-F 6 "" V 3350 1250 60  0001 C CNN "Part Number"
+F 5 "100 mW " V 3350 1250 60  0001 C CNN "Power"
+F 6 "CR0603-F/-9R10ELF" V 3350 1250 60  0001 C CNN "Part Number"
 	1    3350 1250
 	-1   0    0    1
@@
 AR Path="/6366AF3A/63D3885E/63C11627" Ref="R?"  Part="1"
 AR Path="/6366AF3A/63D47A03/63C11627" Ref="R?"  Part="1"
-F 0 "R74" V 3430 1950 50  0000 C CNN
+F 0 "R44" V 3430 1950 50  0000 C CNN
 F 1 "9.1" V 3350 1950 50  0000 C CNN
-F 2 "Resistors_SMD:R_0603_HandSoldering" V 3280 1950 50  0001 C CNN
-F 3 "" H 3350 1950 50  0001 C CNN
+F 2 "Resistors_SMD:R_0603" V 3280 1950 50  0001 C CNN
+F 3 "https://www.mouser.co.il/ProductDetail/Bourns/CR0603-F-9R10ELF?qs=W%2FMpXkg%252BdQ6lipKjUosapQ%3D%3D" H 3350 1950 50  0001 C CNN
 F 4 "1%" V 3350 1950 60  0001 C CNN "Tolerance"
-F 5 "250 mW" V 3350 1950 60  0001 C CNN "Power"
-F 6 "" V 3350 1950 60  0001 C CNN "Part Number"
+F 5 "100 mW " V 3350 1950 60  0001 C CNN "Power"
+F 6 "CR0603-F/-9R10ELF" V 3350 1950 60  0001 C CNN "Part Number"
 	1    3350 1950
 	-1   0    0    1

Commit message: good, before FMC lines connect
Changed lines of the file:
@@
 $Descr A4 11693 8268
 encoding utf-8
-Sheet 5 12
+Sheet 8 12
 Title ""
 Date ""
@@
 AR Path="/6366AF3A/63D3885E/5955E861" Ref="R?"  Part="1"
 AR Path="/6366AF3A/63D47A03/5955E861" Ref="R?"  Part="1"
-F 0 "R39" V 2680 1250 50  0000 C CNN
+F 0 "R57" V 2680 1250 50  0000 C CNN
 F 1 "220" V 2600 1250 50  0000 C CNN
 F 2 "Resistors_SMD:R_0603" V 2530 1250 50  0001 C CNN
@@
 AR Path="/6366AF3A/63D3885E/5955F5C4" Ref="R?"  Part="1"
 AR Path="/6366AF3A/63D47A03/5955F5C4" Ref="R?"  Part="1"
-F 0 "R42" V 2980 1700 50  0000 C CNN
+F 0 "R60" V 2980 1700 50  0000 C CNN
 F 1 "47" V 2900 1700 50  0000 C CNN
 F 2 "Resistors_SMD:R_0603" V 2830 1700 50  0001 C CNN
@@
 AR Path="/6366AF3A/63D3885E/61C6D193" Ref="#PWR?"  Part="1"
 AR Path="/6366AF3A/63D47A03/61C6D193" Ref="#PWR?"  Part="1"
-F 0 "#PWR0117" H 3600 2050 50  0001 C CNN
+F 0 "#PWR0123" H 3600 2050 50  0001 C CNN
 F 1 "Earth" H 3600 2150 50  0001 C CNN
 F 2 "" H 3600 2300 50  0000 C CNN
@@
 AR Path="/6366AF3A/63D3885E/61C6D191" Ref="#PWR?"  Part="1"
 AR Path="/6366AF3A/63D47A03/61C6D191" Ref="#PWR?"  Part="1"
-F 0 "#PWR0118" H 3600 900 50  0001 C CNN
+F 0 "#PWR0124" H 3600 900 50  0001 C CNN
 F 1 "Earth" H 3600 1000 50  0001 C CNN
 F 2 "" H 3600 1150 50  0000 C CNN
@@
 AR Path="/6366AF3A/63D3885E/61C6D194" Ref="R?"  Part="1"
 AR Path="/6366AF3A/63D47A03/61C6D194" Ref="R?"  Part="1"
-F 0 "R40" V 2680 1950 50  0000 C CNN
+F 0 "R58" V 2680 1950 50  0000 C CNN
 F 1 "220" V 2600 1950 50  0000 C CNN
 F 2 "Resistors_SMD:R_0603" V 2530 1950 50  0001 C CNN
@@
 AR Path="/6366AF3A/63D3885E/61C6D195" Ref="R?"  Part="1"
 AR Path="/6366AF3A/63D47A03/61C6D195" Ref="R?"  Part="1"
-F 0 "R41" V 2980 1500 50  0000 C CNN
+F 0 "R59" V 2980 1500 50  0000 C CNN
 F 1 "47" V 2900 1500 50  0000 C CNN
 F 2 "Resistors_SMD:R_0603" V 2830 1500 50  0001 C CNN
@@
 AR Path="/6366AF3A/63D3885E/5955E920" Ref="R?"  Part="1"
 AR Path="/6366AF3A/63D47A03/5955E920" Ref="R?"  Part="1"
-F 0 "R43" V 3430 1250 50  0000 C CNN
+F 0 "R61" V 3430 1250 50  0000 C CNN
 F 1 "9.1" V 3350 1250 50  0000 C CNN
 F 2 "Resistors_SMD:R_0603" V 3280 1250 50  0001 C CNN
@@
 AR Path="/6366AF3A/63D3885E/63C11627" Ref="R?"  Part="1"
 AR Path="/6366AF3A/63D47A03/63C11627" Ref="R?"  Part="1"
-F 0 "R44" V 3430 1950 50  0000 C CNN
+F 0 "R62" V 3430 1950 50  0000 C CNN
 F 1 "9.1" V 3350 1950 50  0000 C CNN
 F 2 "Resistors_SMD:R_0603" V 3280 1950 50  0001 C CNN

Commit message: started routing
Changed lines of the file:
@@
 $Descr A4 11693 8268
 encoding utf-8
-Sheet 8 12
+Sheet 9 12
 Title ""
 Date ""
@@
 AR Path="/6366AF3A/63D3885E/5955E861" Ref="R?"  Part="1"
 AR Path="/6366AF3A/63D47A03/5955E861" Ref="R?"  Part="1"
-F 0 "R57" V 2680 1250 50  0000 C CNN
+F 0 "R63" V 2680 1250 50  0000 C CNN
 F 1 "220" V 2600 1250 50  0000 C CNN
 F 2 "Resistors_SMD:R_0603" V 2530 1250 50  0001 C CNN
@@
 AR Path="/6366AF3A/63D3885E/5955F5C4" Ref="R?"  Part="1"
 AR Path="/6366AF3A/63D47A03/5955F5C4" Ref="R?"  Part="1"
-F 0 "R60" V 2980 1700 50  0000 C CNN
+F 0 "R66" V 2980 1700 50  0000 C CNN
 F 1 "47" V 2900 1700 50  0000 C CNN
 F 2 "Resistors_SMD:R_0603" V 2830 1700 50  0001 C CNN
@@
 AR Path="/6366AF3A/63D3885E/61C6D194" Ref="R?"  Part="1"
 AR Path="/6366AF3A/63D47A03/61C6D194" Ref="R?"  Part="1"
-F 0 "R58" V 2680 1950 50  0000 C CNN
+F 0 "R64" V 2680 1950 50  0000 C CNN
 F 1 "220" V 2600 1950 50  0000 C CNN
 F 2 "Resistors_SMD:R_0603" V 2530 1950 50  0001 C CNN
@@
 AR Path="/6366AF3A/63D3885E/61C6D195" Ref="R?"  Part="1"
 AR Path="/6366AF3A/63D47A03/61C6D195" Ref="R?"  Part="1"
-F 0 "R59" V 2980 1500 50  0000 C CNN
+F 0 "R65" V 2980 1500 50  0000 C CNN
 F 1 "47" V 2900 1500 50  0000 C CNN
 F 2 "Resistors_SMD:R_0603" V 2830 1500 50  0001 C CNN
@@
 AR Path="/6366AF3A/63D3885E/5955E920" Ref="R?"  Part="1"
 AR Path="/6366AF3A/63D47A03/5955E920" Ref="R?"  Part="1"
-F 0 "R61" V 3430 1250 50  0000 C CNN
+F 0 "R67" V 3430 1250 50  0000 C CNN
 F 1 "9.1" V 3350 1250 50  0000 C CNN
 F 2 "Resistors_SMD:R_0603" V 3280 1250 50  0001 C CNN
@@
 AR Path="/6366AF3A/63D3885E/63C11627" Ref="R?"  Part="1"
 AR Path="/6366AF3A/63D47A03/63C11627" Ref="R?"  Part="1"
-F 0 "R62" V 3430 1950 50  0000 C CNN
+F 0 "R68" V 3430 1950 50  0000 C CNN
 F 1 "9.1" V 3350 1950 50  0000 C CNN
 F 2 "Resistors_SMD:R_0603" V 3280 1950 50  0001 C CNN

Commit message: before hi-speed routing
Other:
- note added: "NOTE: Every such block consumes around 20mA.\n\nFor 18 blocks (Six (6) 2 lanes CSI + 6 clocks) = 6*2 + 6 = 18 we need 18*0.02A = 0.36 A ,around 0.5 A\n---------------------------------------------------------\n\n\nFor 6 blocks we need 6*0.02A = 0.12 A = 0.12*2.5 = 0.3 Watt"
- note removed: "NOTE: Every such block consumes around 20mA.\n\nFor 18 blocks (Six (6) 2 lanes CSI + 6 clocks) = 6*2 + 6 = 18 we need 18*0.02A = 0.36 A ,around 0.5 A"
Changed lines of the file:
@@
 $Descr A4 11693 8268
 encoding utf-8
-Sheet 9 12
+Sheet 10 12
 Title ""
 Date ""
@@
 AR Path="/6366AF3A/63D3885E/5955E861" Ref="R?"  Part="1"
 AR Path="/6366AF3A/63D47A03/5955E861" Ref="R?"  Part="1"
-F 0 "R63" V 2680 1250 50  0000 C CNN
+F 0 "R69" V 2680 1250 50  0000 C CNN
 F 1 "220" V 2600 1250 50  0000 C CNN
 F 2 "Resistors_SMD:R_0603" V 2530 1250 50  0001 C CNN
@@
 AR Path="/6366AF3A/63D3885E/5955F5C4" Ref="R?"  Part="1"
 AR Path="/6366AF3A/63D47A03/5955F5C4" Ref="R?"  Part="1"
-F 0 "R66" V 2980 1700 50  0000 C CNN
+F 0 "R72" V 2980 1700 50  0000 C CNN
 F 1 "47" V 2900 1700 50  0000 C CNN
 F 2 "Resistors_SMD:R_0603" V 2830 1700 50  0001 C CNN
@@
 AR Path="/6366AF3A/63D3885E/61C6D194" Ref="R?"  Part="1"
 AR Path="/6366AF3A/63D47A03/61C6D194" Ref="R?"  Part="1"
-F 0 "R64" V 2680 1950 50  0000 C CNN
+F 0 "R70" V 2680 1950 50  0000 C CNN
 F 1 "220" V 2600 1950 50  0000 C CNN
 F 2 "Resistors_SMD:R_0603" V 2530 1950 50  0001 C CNN
@@
 AR Path="/6366AF3A/63D3885E/61C6D195" Ref="R?"  Part="1"
 AR Path="/6366AF3A/63D47A03/61C6D195" Ref="R?"  Part="1"
-F 0 "R65" V 2980 1500 50  0000 C CNN
+F 0 "R71" V 2980 1500 50  0000 C CNN
 F 1 "47" V 2900 1500 50  0000 C CNN
 F 2 "Resistors_SMD:R_0603" V 2830 1500 50  0001 C CNN
@@
 AR Path="/6366AF3A/63D3885E/5955E920" Ref="R?"  Part="1"
 AR Path="/6366AF3A/63D47A03/5955E920" Ref="R?"  Part="1"
-F 0 "R67" V 3430 1250 50  0000 C CNN
+F 0 "R73" V 3430 1250 50  0000 C CNN
 F 1 "9.1" V 3350 1250 50  0000 C CNN
 F 2 "Resistors_SMD:R_0603" V 3280 1250 50  0001 C CNN
@@
 AR Path="/6366AF3A/63D3885E/63C11627" Ref="R?"  Part="1"
 AR Path="/6366AF3A/63D47A03/63C11627" Ref="R?"  Part="1"
-F 0 "R68" V 3430 1950 50  0000 C CNN
+F 0 "R74" V 3430 1950 50  0000 C CNN
 F 1 "9.1" V 3350 1950 50  0000 C CNN
 F 2 "Resistors_SMD:R_0603" V 3280 1950 50  0001 C CNN
@@
 $EndComp
 Text Notes 1100 3000 0    79   ~ 16
-NOTE: Every such block consumes around 20mA.\n\nFor 18 blocks (Six (6) 2 lanes CSI + 6 clocks) = 6*2 + 6 = 18 we need 18*0.02A = 0.36 A ,around 0.5 A
+NOTE: Every such block consumes around 20mA.\n\nFor 18 blocks (Six (6) 2 lanes CSI + 6 clocks) = 6*2 + 6 = 18 we need 18*0.02A = 0.36 A ,around 0.5 A\n---------------------------------------------------------\n\n\nFor 6 blocks  we need 6*0.02A = 0.12 A = 0.12*2.5 = 0.3 Watt
 $EndSCHEMATC
