File: LVDS_2_SLVS.kicad_sch (KiCad schematic)
At the start: 6 parts

Commit message: DRC, ERC OK
Parts:
- R45, R46, R47, R48, R49, R50: symbol FMC_MIPI_v2-rescue:R-Device -> FMC_MIPI_v2:R
Changed lines of the file:
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@@
     (effects (font (size 1.27 1.27)) (justify right))
   )
-  (symbol (lib_id "FMC_MIPI_v2-rescue:R-Device") (at 66.04 31.75 180) (unit 1)
+  (symbol (lib_id "FMC_MIPI_v2:R") (at 66.04 31.75 180) (unit 1)
     (in_bom yes) (on_board yes)
     (property "Reference" "R46" (id 0) (at 64.008 31.75 90))
@@
     (pin "2")
   )
-  (symbol (lib_id "FMC_MIPI_v2-rescue:R-Device") (at 85.09 31.75 180) (unit 1)
+  (symbol (lib_id "FMC_MIPI_v2:R") (at 85.09 31.75 180) (unit 1)
     (in_bom yes) (on_board yes)
     (property "Reference" "R50" (id 0) (at 83.058 31.75 90))
@@
     (pin "2")
   )
-  (symbol (lib_id "FMC_MIPI_v2-rescue:R-Device") (at 73.66 43.18 270) (mirror x) (unit 1)
+  (symbol (lib_id "FMC_MIPI_v2:R") (at 73.66 43.18 270) (mirror x) (unit 1)
     (in_bom yes) (on_board yes)
     (property "Reference" "R47" (id 0) (at 73.66 41.148 90))
@@
     (pin "1")
   )
-  (symbol (lib_id "FMC_MIPI_v2-rescue:R-Device") (at 66.04 49.53 180) (unit 1)
+  (symbol (lib_id "FMC_MIPI_v2:R") (at 66.04 49.53 180) (unit 1)
     (in_bom yes) (on_board yes)
     (property "Reference" "R45" (id 0) (at 64.008 49.53 90))
@@
     (pin "2")
   )
-  (symbol (lib_id "FMC_MIPI_v2-rescue:R-Device") (at 73.66 38.1 270) (mirror x) (unit 1)
+  (symbol (lib_id "FMC_MIPI_v2:R") (at 73.66 38.1 270) (mirror x) (unit 1)
     (in_bom yes) (on_board yes)
     (property "Reference" "R48" (id 0) (at 73.66 36.068 90))
@@
     (pin "2")
   )
-  (symbol (lib_id "FMC_MIPI_v2-rescue:R-Device") (at 85.09 49.53 180) (unit 1)
+  (symbol (lib_id "FMC_MIPI_v2:R") (at 85.09 49.53 180) (unit 1)
     (in_bom yes) (on_board yes)
     (property "Reference" "R49" (id 0) (at 83.058 49.53 90))

Commit message: JLCPCB BOM OK
Parts:
- R45, R46: LCSC (none) -> C107696
- R47, R48: LCSC (none) -> C114623
- R49, R50: LCSC (none) -> C103890
Changed lines of the file:
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@@
       (effects (font (size 1.524 1.524)) hide)
+    )
+    (property "LCSC" "C107696" (id 7) (at 66.04 31.75 90)
+      (effects (font (size 1.27 1.27)) hide)
     )
     (pin "1")
@@
       (effects (font (size 1.524 1.524)) hide)
     )
+    (property "LCSC" "C103890" (id 7) (at 85.09 31.75 90)
+      (effects (font (size 1.27 1.27)) hide)
+    )
     (pin "1")
     (pin "2")
@@
     (property "Part Number" "RC0603FR-0747RL" (id 6) (at 73.66 43.18 90)
       (effects (font (size 1.524 1.524)) hide)
+    )
+    (property "LCSC" "C114623" (id 7) (at 73.66 43.18 90)
+      (effects (font (size 1.27 1.27)) hide)
     )
     (pin "1")
@@
       (effects (font (size 1.524 1.524)) hide)
     )
+    (property "LCSC" "C107696" (id 7) (at 66.04 49.53 90)
+      (effects (font (size 1.27 1.27)) hide)
+    )
     (pin "1")
     (pin "2")
@@
     (property "Part Number" "RC0603FR-0747RL" (id 6) (at 73.66 38.1 90)
       (effects (font (size 1.524 1.524)) hide)
+    )
+    (property "LCSC" "C114623" (id 7) (at 73.66 38.1 90)
+      (effects (font (size 1.27 1.27)) hide)
     )
     (pin "1")
@@
       (effects (font (size 1.524 1.524)) hide)
     )
+    (property "LCSC" "C103890" (id 7) (at 85.09 49.53 90)
+      (effects (font (size 1.27 1.27)) hide)
+    )
     (pin "1")
